File: HB_Drive_V1/DeadTime.kicad_sch (KiCad schematic)
At the start: 15 parts, among them J4 Conn_01x02, J5 Conn_01x02, U5 74LS08, U6 74AUC2G02, U7 74LS08, U8 74LS365

Commit message: finishes hirearchical labels, add 10v +- ref generation and updates the DC offset circuits
Parts:
- renumbered C40 to C19, C41 to C20, C12 to C21, C13 to C22, C14 to C23, J4 to J7, J5 to J8, R72 to R52, R75 to R53, R30 to R54, R31 to R55, U6 to U10, U8 to U11, U7 to U12, U5 to U9
