File: HB_Drive_V1/Comparator.kicad_sch (KiCad schematic)
At the start: 9 parts, among them J6 Conn_02x02_Odd_Even, U9 LM311

Commit message: finishes hirearchical labels, add 10v +- ref generation and updates the DC offset circuits
Parts:
- renumbered C15 to C24, C16 to C25, C17 to C26, J6 to J9, R32 to R56, R33 to R57, R34 to R58, TP6 to TP11, U9 to U13
Changed lines of the file:
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@@
 		(in_pos_files yes)
 		(dnp no)
-		(property "Reference" "C17"
+		(property "Reference" "C26"
 			(at 168.91 101.6 90)
 			(hide yes)
@@
 			(project "HB_Drive_V1"
 				(path "/a9b54c89-4c8e-4c90-8a0d-ec2009e369b7/28e2d9d3-ebce-4623-8c7e-52f93025d826/ddec5c9b-01ea-44af-a206-8cb280d1ab2e"
-					(reference "C17")
+					(reference "C26")
 					(unit 1)
 				)
@@
 		(in_pos_files yes)
 		(dnp no)
-		(property "Reference" "#PWR031"
+		(property "Reference" "#PWR059"
 			(at 138.43 85.09 0)
 			(hide yes)
@@
 			(project "HB_Drive_V1"
 				(path "/a9b54c89-4c8e-4c90-8a0d-ec2009e369b7/28e2d9d3-ebce-4623-8c7e-52f93025d826/ddec5c9b-01ea-44af-a206-8cb280d1ab2e"
-					(reference "#PWR031")
+					(reference "#PWR059")
 					(unit 1)
 				)
@@
 		(dnp no)
 		(fields_autoplaced yes)
-		(property "Reference" "#PWR036"
+		(property "Reference" "#PWR064"
 			(at 163.83 95.25 0)
 			(hide yes)
@@
 			(project "HB_Drive_V1"
 				(path "/a9b54c89-4c8e-4c90-8a0d-ec2009e369b7/28e2d9d3-ebce-4623-8c7e-52f93025d826/ddec5c9b-01ea-44af-a206-8cb280d1ab2e"
-					(reference "#PWR036")
+					(reference "#PWR064")
 					(unit 1)
 				)
@@
 		(in_pos_files yes)
 		(dnp no)
-		(property "Reference" "C15"
+		(property "Reference" "C24"
 			(at 147.32 76.2 90)
 			(hide yes)
@@
 			(project "HB_Drive_V1"
 				(path "/a9b54c89-4c8e-4c90-8a0d-ec2009e369b7/28e2d9d3-ebce-4623-8c7e-52f93025d826/ddec5c9b-01ea-44af-a206-8cb280d1ab2e"
-					(reference "C15")
+					(reference "C24")
 					(unit 1)
 				)
@@
 		(in_pos_files yes)
 		(dnp no)
-		(property "Reference" "#PWR033"
+		(property "Reference" "#PWR061"
 			(at 153.67 77.47 0)
 			(hide yes)
@@
 			(project "HB_Drive_V1"
 				(path "/a9b54c89-4c8e-4c90-8a0d-ec2009e369b7/28e2d9d3-ebce-4623-8c7e-52f93025d826/ddec5c9b-01ea-44af-a206-8cb280d1ab2e"
-					(reference "#PWR033")
+					(reference "#PWR061")
 					(unit 1)
 				)
@@
 		(in_pos_files yes)
 		(dnp no)
-		(property "Reference" "TP6"
+		(property "Reference" "TP11"
 			(at 165.862 82.296 0)
 			(show_name no)
@@
 			(project "HB_Drive_V1"
 				(path "/a9b54c89-4c8e-4c90-8a0d-ec2009e369b7/28e2d9d3-ebce-4623-8c7e-52f93025d826/ddec5c9b-01ea-44af-a206-8cb280d1ab2e"
-					(reference "TP6")
+					(reference "TP11")
 					(unit 1)
 				)
@@
 		(in_pos_files yes)
 		(dnp no)
-		(property "Reference" "#PWR032"
+		(property "Reference" "#PWR060"
 			(at 138.43 109.22 0)
 			(hide yes)
@@
 			(project "HB_Drive_V1"
 				(path "/a9b54c89-4c8e-4c90-8a0d-ec2009e369b7/28e2d9d3-ebce-4623-8c7e-52f93025d826/ddec5c9b-01ea-44af-a206-8cb280d1ab2e"
-					(reference "#PWR032")
+					(reference "#PWR060")
 					(unit 1)
 				)
@@
 		(in_pos_files yes)
 		(dnp no)
-		(property "Reference" "R33"
+		(property "Reference" "R57"
 			(at 133.35 88.9 90)
 			(hide yes)
@@
 			(project "HB_Drive_V1"
 				(path "/a9b54c89-4c8e-4c90-8a0d-ec2009e369b7/28e2d9d3-ebce-4623-8c7e-52f93025d826/ddec5c9b-01ea-44af-a206-8cb280d1ab2e"
-					(reference "R33")
+					(reference "R57")
 					(unit 1)
 				)
@@
 		(in_pos_files yes)
 		(dnp no)
-		(property "Reference" "C16"
+		(property "Reference" "C25"
 			(at 147.32 96.52 90)
 			(hide yes)
@@
 			(project "HB_Drive_V1"
 				(path "/a9b54c89-4c8e-4c90-8a0d-ec2009e369b7/28e2d9d3-ebce-4623-8c7e-52f93025d826/ddec5c9b-01ea-44af-a206-8cb280d1ab2e"
-					(reference "C16")
+					(reference "C25")
 					(unit 1)
 				)
@@
 		(in_pos_files yes)
 		(dnp no)
-		(property "Reference" "U9"
+		(property "Reference" "U13"
 			(at 160.782 90.932 0)
 			(show_name no)
@@
 			(project "HB_Drive_V1"
 				(path "/a9b54c89-4c8e-4c90-8a0d-ec2009e369b7/28e2d9d3-ebce-4623-8c7e-52f93025d826/ddec5c9b-01ea-44af-a206-8cb280d1ab2e"
-					(reference "U9")
+					(reference "U13")
 					(unit 1)
 				)
@@
 		(in_pos_files yes)
 		(dnp no)
-		(property "Reference" "#PWR035"
+		(property "Reference" "#PWR063"
 			(at 156.21 109.22 0)
 			(hide yes)
@@
 			(project "HB_Drive_V1"
 				(path "/a9b54c89-4c8e-4c90-8a0d-ec2009e369b7/28e2d9d3-ebce-4623-8c7e-52f93025d826/ddec5c9b-01ea-44af-a206-8cb280d1ab2e"
-					(reference "#PWR035")
+					(reference "#PWR063")
 					(unit 1)
 				)
@@
 		(in_pos_files yes)
 		(dnp no)
-		(property "Reference" "#PWR034"
+		(property "Reference" "#PWR062"
 			(at 153.67 99.06 0)
 			(hide yes)
@@
 			(project "HB_Drive_V1"
 				(path "/a9b54c89-4c8e-4c90-8a0d-ec2009e369b7/28e2d9d3-ebce-4623-8c7e-52f93025d826/ddec5c9b-01ea-44af-a206-8cb280d1ab2e"
-					(reference "#PWR034")
+					(reference "#PWR062")
 					(unit 1)
 				)
@@
 		(in_pos_files yes)
 		(dnp no)
-		(property "Reference" "#PWR037"
+		(property "Reference" "#PWR065"
 			(at 167.64 109.22 0)
 			(hide yes)
@@
 			(project "HB_Drive_V1"
 				(path "/a9b54c89-4c8e-4c90-8a0d-ec2009e369b7/28e2d9d3-ebce-4623-8c7e-52f93025d826/ddec5c9b-01ea-44af-a206-8cb280d1ab2e"
-					(reference "#PWR037")
+					(reference "#PWR065")
 					(unit 1)
 				)
@@
 		(in_pos_files yes)
 		(dnp no)
-		(property "Reference" "R34"
+		(property "Reference" "R58"
 			(at 168.91 95.25 90)
 			(hide yes)
@@
 			(project "HB_Drive_V1"
 				(path "/a9b54c89-4c8e-4c90-8a0d-ec2009e369b7/28e2d9d3-ebce-4623-8c7e-52f93025d826/ddec5c9b-01ea-44af-a206-8cb280d1ab2e"
-					(reference "R34")
+					(reference "R58")
 					(unit 1)
 				)
@@
 		(in_pos_files yes)
 		(dnp no)
-		(property "Reference" "J6"
+		(property "Reference" "J9"
 			(at 118.11 82.55 0)
 			(show_name no)
@@
 			(project "HB_Drive_V1"
 				(path "/a9b54c89-4c8e-4c90-8a0d-ec2009e369b7/28e2d9d3-ebce-4623-8c7e-52f93025d826/ddec5c9b-01ea-44af-a206-8cb280d1ab2e"
-					(reference "J6")
+					(reference "J9")
 					(unit 1)
 				)
@@
 		(in_pos_files yes)
 		(dnp no)
-		(property "Reference" "R32"
+		(property "Reference" "R56"
 			(at 133.35 83.82 90)
 			(hide yes)
@@
 			(project "HB_Drive_V1"
 				(path "/a9b54c89-4c8e-4c90-8a0d-ec2009e369b7/28e2d9d3-ebce-4623-8c7e-52f93025d826/ddec5c9b-01ea-44af-a206-8cb280d1ab2e"
-					(reference "R32")
-					(unit 1)
-				)
+					(reference "R56")
+					(unit 1)
+				)

Commit message: updates board to highest working copy
Parts:
- removed J9: Conn_02x02_Odd_Even, Connector_PinSocket_1.27mm:PinSocket_2x02_P1.27mm_Vertical, symbol Connector_Generic:Conn_02x02_Odd_Even
- removed R58: 1KΩ, Resistor_SMD:R_0603_1608Metric_Pad0.98x0.95mm_HandSolder, symbol Device:R_Small_US
- added R603: 1KΩ, Resistor_SMD:R_0603_1608Metric_Pad0.98x0.95mm_HandSolder, symbol Device:R_Small_US
- renumbered C24 to C601, C25 to C602, C26 to C603, R56 to R601, R57 to R602, TP11 to TP601, U13 to U601
Connections:
- net +5V: now also R603.2
- net Carrier: now also R602.1
- net D_Cmd: now also R601.1
- net H_Cmd: now also R603.1
Other:
- moved on the sheet: TP601, U601
