File: HB_Drive_V1/HB_Drive_V1.kicad_pcb (KiCad board)
At the start: 2 copper layers, 156 parts, among them J1 Conn_02x05_Counter_Clockwise, J11 Conn_02x03_Counter_Clockwise, J12 Conn_01x02, J2 Conn_02x03_Counter_Clockwise, J3 Conn_01x02, J4 Conn_01x02, J5 Conn_01x02, J6 Conn_02x02_Odd_Even, J7 Conn_02x04_Counter_Clockwise, U1 TL082, U10 NE555D, U11 TL082, U12 TL082, U13 TL082, U15 TL082, U19 74LS32, U3 TL082, U4 TL082

Commit message: finishes hirearchical labels, add 10v +- ref generation and updates the DC offset circuits
Parts:
- removed J11: Conn_02x03_Counter_Clockwise, Connector_PinSocket_1.27mm:PinSocket_2x03_P1.27mm_Vertical
- removed J12: Conn_01x02, Connector_PinHeader_1.27mm:PinHeader_1x02_P1.27mm_Vertical
- removed the R51 at (174.5, 110.3)
- removed the R53 at (218.0, 67.9)
- removed the R54 at (218.0, 70.4)
- removed the R55 at (218.0, 73.0)
- removed the R56 at (218.0, 75.5)
- removed the R57 at (222.4, 65.4)
- removed the R70 at (226.7, 65.4)
- removed the R71 at (226.7, 67.9)
- removed the R73 at (226.7, 70.4)
- removed the R74 at (207.7, 65.5)
- removed the R9 at (113.2, 88.9)
- removed the TP15 at (177.2, 86.9)
- removed the TP21 at (218.4, 61.6)
- removed U13: TL082, Package_SO:SOIC-8_5.3x5.3mm_P1.27mm
- added C1: 100nF 100V, Capacitor_SMD:C_0603_1608Metric, F.Cu at (72.2, 43.6)
- added C2: 100nF 100V, Capacitor_SMD:C_0603_1608Metric, F.Cu at (72.2, 46.1)
- added C27: 1uF, Capacitor_SMD:C_0603_1608Metric, F.Cu at (97.0, 55.3)
- added C4: 100nF 100V, Capacitor_SMD:C_0603_1608Metric, F.Cu at (72.2, 48.6)
- added C48: 10nF, Capacitor_SMD:C_0603_1608Metric_Pad1.08x0.95mm_HandSolder, F.Cu at (83.8, 72.4)
- added C49: 10nF, Capacitor_SMD:C_0603_1608Metric_Pad1.08x0.95mm_HandSolder, F.Cu at (83.8, 74.9)
- added C5: 100nF 100V, Capacitor_SMD:C_0603_1608Metric, F.Cu at (72.2, 51.1)
- added C6: 100nF 100V, Capacitor_SMD:C_0603_1608Metric, F.Cu at (72.2, 53.7)
- added C7: 100nF 100V, Capacitor_SMD:C_0603_1608Metric, F.Cu at (72.2, 56.2)
- added D5: 1N4148W, Diode_SMD:D_SOD-123, F.Cu at (88.9, 72.8)
- added D6: 1N4148W, Diode_SMD:D_SOD-123, F.Cu at (88.9, 76.2)
- added J2: Conn_02x02_Odd_Even, Connector_PinSocket_1.27mm:PinSocket_2x02_P1.27mm_Vertical, F.Cu at (82.6, 66.2)
- added J3: Conn_01x02, Connector_PinHeader_1.27mm:PinHeader_1x02_P1.27mm_Vertical, F.Cu at (77.3, 66.2)
- added J4: Conn_02x05_Counter_Clockwise, Connector_PinHeader_1.27mm:PinHeader_2x05_P1.27mm_Vertical, F.Cu at (74.0, 86.0)
- added R11: 51KΩ, Resistor_SMD:R_0603_1608Metric_Pad0.98x0.95mm_HandSolder, F.Cu at (76.4, 56.2)
- added R12: 10KΩ, Resistor_SMD:R_0603_1608Metric_Pad0.98x0.95mm_HandSolder, F.Cu at (80.8, 43.6)
- added R13: 51KΩ, Resistor_SMD:R_0603_1608Metric_Pad0.98x0.95mm_HandSolder, F.Cu at (80.8, 46.1)
- added R14: PV36W104C01B00, PV36W104C01B00:POT_PV36W_BRN, F.Cu at (62.1, 52.2)
- added R15: 10kΩ, Resistor_SMD:R_0603_1608Metric_Pad0.98x0.95mm_HandSolder, F.Cu at (80.8, 48.6)
- added R16: 10K, Resistor_SMD:R_0603_1608Metric_Pad0.98x0.95mm_HandSolder, F.Cu at (80.8, 51.1)
- added R17: 10kΩ, Resistor_SMD:R_0603_1608Metric_Pad0.98x0.95mm_HandSolder, F.Cu at (80.8, 53.7)
- added R18: PV36W104C01B00, PV36W104C01B00:POT_PV36W_BRN, F.Cu at (62.1, 58.8)
- added R28: 10kΩ, Resistor_SMD:R_0603_1608Metric_Pad0.98x0.95mm_HandSolder, F.Cu at (59.4, 72.4)
- added R29: 10K, Resistor_SMD:R_0603_1608Metric_Pad0.98x0.95mm_HandSolder, F.Cu at (59.4, 74.9)
- added R30: 10K, Resistor_SMD:R_0603_1608Metric_Pad0.98x0.95mm_HandSolder, F.Cu at (59.4, 77.4)
- added R31: 10K, Resistor_SMD:R_0603_1608Metric_Pad0.98x0.95mm_HandSolder, F.Cu at (59.4, 79.9)
- added R32: 10K, Resistor_SMD:R_0603_1608Metric_Pad0.98x0.95mm_HandSolder, F.Cu at (59.4, 82.4)
- added R36: PV36W104C01B00, PV36W104C01B00:POT_PV36W_BRN, F.Cu at (66.4, 74.4)
- added R4: 10kΩ, Resistor_SMD:R_0603_1608Metric_Pad0.98x0.95mm_HandSolder, F.Cu at (76.4, 43.6)
- added R40: 51KΩ, Resistor_SMD:R_0603_1608Metric_Pad0.98x0.95mm_HandSolder, F.Cu at (59.4, 85.0)
- added R41: 51KΩ, Resistor_SMD:R_0603_1608Metric_Pad0.98x0.95mm_HandSolder, F.Cu at (59.4, 87.5)
- added R43: 10KΩ, Resistor_SMD:R_0603_1608Metric_Pad0.98x0.95mm_HandSolder, F.Cu at (59.4, 90.0)
- added R45: 51KΩ, Resistor_SMD:R_0603_1608Metric_Pad0.98x0.95mm_HandSolder, F.Cu at (59.4, 92.5)
- added R46: PV36W104C01B00, PV36W104C01B00:POT_PV36W_BRN, F.Cu at (66.4, 81.0)
- added R5: 10K, Resistor_SMD:R_0603_1608Metric_Pad0.98x0.95mm_HandSolder, F.Cu at (76.4, 46.1)
- added R59: PV36W104C01B00, PV36W104C01B00:POT_PV36W_BRN, F.Cu at (91.4, 45.6)
- added R85: 680Ω, Resistor_SMD:R_0603_1608Metric_Pad0.98x0.95mm_HandSolder, F.Cu at (83.8, 77.4)
- added R86: PV36W103C01B00, PV36W104C01B00:POT_PV36W_BRN, F.Cu at (90.9, 81.1)
- added R87: 1KΩ, Resistor_SMD:R_0603_1608Metric_Pad0.98x0.95mm_HandSolder, F.Cu at (83.8, 79.9)
- added TP1: TestPoint, TestPoint:TestPoint_Loop_D2.60mm_Drill1.6mm_Beaded, F.Cu at (72.7, 59.9)
- added TP12: TestPoint, TestPoint:TestPoint_Loop_D2.60mm_Drill1.6mm_Beaded, F.Cu at (97.5, 51.5)
- added TP2: TestPoint, TestPoint:TestPoint_Loop_D2.60mm_Drill1.6mm_Beaded, F.Cu at (72.7, 65.0)
- added TP9: TestPoint, TestPoint:TestPoint_Loop_D2.60mm_Drill1.6mm_Beaded, F.Cu at (77.1, 73.7)
- added U14: REF102CU, Package_SO:SOIC-8_3.9x4.9mm_P1.27mm, F.Cu at (90.7, 52.3)
- added U2: TL082, Package_SO:SOIC-8_5.3x5.3mm_P1.27mm, F.Cu at (62.4, 65.7)
- added U21: NE555D, Package_SO:SOIC-8_3.9x4.9mm_P1.27mm, F.Cu at (96.0, 74.5)
- added U7: TL082, Package_SO:SOIC-8_5.3x5.3mm_P1.27mm, F.Cu at (66.7, 87.9)
- J1: value Conn_02x05_Counter_Clockwise -> Conn_02x04_Counter_Clockwise; footprint Connector_PinHeader_1.27mm:PinHeader_2x05_P1.27mm_Vertical -> Connector_PinSocket_1.27mm:PinSocket_2x04_P1.27mm_Vertical
- R10: value 10K -> 51KΩ
- R6: value 10kΩ -> 10K
- R8: value 10K -> PV36W104C01B00; footprint Resistor_SMD:R_0603_1608Metric_Pad0.98x0.95mm_HandSolder -> PV36W104C01B00:POT_PV36W_BRN
- moved R6 110.6 mm to (76.4, 48.6)
- moved R8 65.4 mm to (62.1, 45.6)
- moved J1 63.6 mm to (78.5, 59.1)
- moved R10 52.7 mm to (76.4, 53.7)
- moved R7 49.2 mm to (76.4, 51.1)
- renumbered C3 to C10, C4 to C11, C5 to C12, C6 to C13, C7 to C14, C8 to C15, C9 to C16, C10 to C17, C11 to C18, C40 to C19, C41 to C20, C12 to C21, C13 to C22, C14 to C23, C15 to C24, C16 to C25, C17 to C26, C36 to C28, C38 to C29, C27 to C3, C37 to C30, C25 to C31, C26 to C32, C28 to C33, C29 to C34, C34 to C35, C35 to C36, C33 to C37, C30 to C38, C31 to C39, C32 to C40, C18 to C41, C19 to C42, C20 to C43, C21 to C44, C22 to C45, C23 to C46, C24 to C47, C1 to C8, C2 to C9, D2 to D1, D3 to D2, D1 to D3, J7 to J10, J2 to J5, J3 to J6, J4 to J7, J5 to J8, J6 to J9, R49 to R1, R59 to R19, R50 to R2, R68 to R20, R69 to R21, R1 to R22, R2 to R23, R3 to R24, R4 to R25, R13 to R26, R5 to R27, R52 to R3, R16 to R33, R11 to R34, R12 to R35, R19 to R37, R14 to R38, R15 to R39, R17 to R42, R18 to R44, R20 to R47, R21 to R48, R22 to R49, R23 to R50, R24 to R51, R72 to R52, R75 to R53, R30 to R54, R31 to R55, R32 to R56, R33 to R57, R34 to R58, R25 to R60, R26 to R61, R27 to R62, R47 to R63, R60 to R64, R61 to R65, R48 to R66, R63 to R68, R62 to R69, R64 to R70, R66 to R71, R65 to R72, R35 to R73, R36 to R74, R37 to R75, R38 to R76, R39 to R77, R40 to R78, R41 to R79, R42 to R80, R43 to R81, R44 to R82, R45 to R83, R46 to R84, R58 to R9, TP5 to TP10, TP6 to TP11, TP11 to TP13, TP13 to TP14, TP20 to TP15, TP7 to TP20, TP8 to TP21, TP9 to TP22, TP10 to TP23, TP12 to TP3, TP14 to TP4, TP2 to TP5, TP1 to TP6, TP3 to TP7, TP4 to TP8, U15 to U1, U19 to U16, U12 to U17, U10 to U19, U11 to U20, U3 to U4, U1 to U5, U4 to U8
Connections:
- net /Outer Voltage Regulator/+I_Err renamed /Outer Voltage Regulator/+V_Err
- J1 pad 1: /INT_AC_REF -> /INT_DC_REF
- J1 pad 2: /INT_DC_REF -> /INT_AC_REF
- J1 pad 4: /Inner Current Regulator/I_Cmd -> /Outer Voltage Regulator/-V_Fdbk
- J1 pad 5: /Inner Current Regulator/-I_Fdbk -> Net-(J1-Pin_5)
- R10 pad 1: Net-(J1-Pin_6) -> Net-(U2A-+)
- R10 pad 2: Net-(U3A--) -> Net-(R10-Pad2)
- R19 pad 2: Net-(U20A--) (its old number) -> /Outer Voltage Regulator/Err_Cmd
- R26 pad 2: Net-(U3A--) -> /Inner Current Regulator/Err_Cmd
- R6 pad 1: Net-(U3A--) -> Net-(J1-Pin_6)
- R6 pad 2: Net-(J1-Pin_10) -> Net-(R10-Pad2)
- R7 pad 1: Net-(J1-Pin_9) -> Net-(J1-Pin_5)
- R7 pad 2: Net-(U3A--) -> Net-(R10-Pad2)
- R8 pad 1: Net-(J1-Pin_8) -> +15V
- R8 pad 2: Net-(U3A--) -> Net-(R11-Pad2)
- U1 pad 4: +15V -> -15V
- U1 pad 8: -15V -> +15V
- U4 pad 2: Net-(U3A--) -> /Inner Current Regulator/Err_Cmd

Commit message: updates board to highest working copy
Parts:
- removed C1, C11, C12, C13, C14, C15, C16, C17, C18, C19, C2, C20, C23, C24, C25, C26, C28, C29, C30, C31, C32, C33, C34, C35, C36, C37, C38, C39, C4, C42, C43, C46, C47, C5, C6, C7: 100nF 100V, Capacitor_SMD:C_0603_1608Metric
- removed C10, C3: 10uF 5%, Capacitor_SMD:C_0603_1608Metric
- removed C21, C22: 470pF 50V, Capacitor_SMD:C_0603_1608Metric
- removed C27: 1uF, Capacitor_SMD:C_0603_1608Metric
- removed C40: 100pF, Capacitor_SMD:C_0603_1608Metric
- removed C41, C44, C45: 100pF 50V, Capacitor_SMD:C_0603_1608Metric
- removed C48, C49: 10nF, Capacitor_SMD:C_0603_1608Metric_Pad1.08x0.95mm_HandSolder
- removed C8, C9: 27uF 5%, Capacitor_SMD:C_0603_1608Metric
- removed D1, D2: MMBD914LT3G, Package_TO_SOT_SMD:SOT-23-3
- removed D3: RED [XL-2012SURC], LED_SMD:LED_0805_2012Metric_Pad1.15x1.40mm_HandSolder
- removed D4: GREEN [XL-2012UGC], LED_SMD:LED_0805_2012Metric_Pad1.15x1.40mm_HandSolder
- removed D5, D6: 1N4148W, Diode_SMD:D_SOD-123
- removed J1, J10: Conn_02x04_Counter_Clockwise, Connector_PinSocket_1.27mm:PinSocket_2x04_P1.27mm_Vertical
- removed J2, J9: Conn_02x02_Odd_Even, Connector_PinSocket_1.27mm:PinSocket_2x02_P1.27mm_Vertical
- removed J3, J6: Conn_01x02, Connector_PinHeader_1.27mm:PinHeader_1x02_P1.27mm_Vertical
- removed J4: Conn_02x05_Counter_Clockwise, Connector_PinHeader_1.27mm:PinHeader_2x05_P1.27mm_Vertical
- removed J5: Conn_02x03_Counter_Clockwise, Connector_PinSocket_1.27mm:PinSocket_2x03_P1.27mm_Vertical
- removed J7, J8: Conn_01x02, Jumper:SolderJumper-2_P1.3mm_Open_TrianglePad1.0x1.5mm
- removed R1, R14, R18, R22, R24, R3, R36, R44, R46, R51, R59, R73, R8, R80, R82: PV36W104C01B00, PV36W104C01B00:POT_PV36W_BRN
- removed R10, R11, R13, R40, R41, R45, R75, R76, R77, R79: 51KΩ, Resistor_SMD:R_0603_1608Metric_Pad0.98x0.95mm_HandSolder
- removed R12, R43, R60, R61, R62, R63, R64, R65, R66, R78, R83: 10KΩ, Resistor_SMD:R_0603_1608Metric_Pad0.98x0.95mm_HandSolder
- removed R15, R17, R19, R20, R21, R26, R28, R33, R37, R4, R47, R50: 10kΩ, Resistor_SMD:R_0603_1608Metric_Pad0.98x0.95mm_HandSolder
- removed R16, R2, R23, R29, R30, R31, R32, R48, R49, R5, R6, R7: 10K, Resistor_SMD:R_0603_1608Metric_Pad0.98x0.95mm_HandSolder
- removed R25: 301kΩ 1%, Resistor_SMD:R_0603_1608Metric_Pad0.98x0.95mm_HandSolder
- removed R27: 10.2kΩ 1%, Resistor_SMD:R_0603_1608Metric_Pad0.98x0.95mm_HandSolder
- removed R34: 976kΩ 1%, Resistor_SMD:R_0603_1608Metric_Pad0.98x0.95mm_HandSolder
- removed R35, R84, R9: 1MΩ 5%, Resistor_SMD:R_0603_1608Metric_Pad0.98x0.95mm_HandSolder
- removed R38: 402kΩ 1%, Resistor_SMD:R_0603_1608Metric_Pad0.98x0.95mm_HandSolder
- removed R39: 6.65kΩ 1%, Resistor_SMD:R_0603_1608Metric_Pad0.98x0.95mm_HandSolder
- removed R42: 10kΩ 1%, Resistor_SMD:R_0603_1608Metric_Pad0.98x0.95mm_HandSolder
- removed R52, R53: PV36W502C01B00, PV36W104C01B00:POT_PV36W_BRN
- removed R54, R55, R81: 100KΩ, Resistor_SMD:R_0603_1608Metric_Pad0.98x0.95mm_HandSolder
- removed R56, R57, R58, R67, R69, R70, R74, R87: 1KΩ, Resistor_SMD:R_0603_1608Metric_Pad0.98x0.95mm_HandSolder
- removed R68: 100Ω, Resistor_SMD:R_0603_1608Metric_Pad0.98x0.95mm_HandSolder
- removed R71, R72: 470Ω, Resistor_SMD:R_0603_1608Metric_Pad0.98x0.95mm_HandSolder
- removed R85: 680Ω, Resistor_SMD:R_0603_1608Metric_Pad0.98x0.95mm_HandSolder
- removed R86: PV36W103C01B00, PV36W104C01B00:POT_PV36W_BRN
- removed TP1, TP10, TP11, TP12, TP13, TP14, TP15, TP16, TP17, TP18, TP19, TP2, TP20, TP21, TP22, TP23, TP3, TP4, TP5, TP6, TP7, TP8, TP9: TestPoint, TestPoint:TestPoint_Loop_D2.60mm_Drill1.6mm_Beaded
- removed U1, U17, U2, U20, U4, U5, U7, U8: TL082, Package_SO:SOIC-8_5.3x5.3mm_P1.27mm
- removed U14: REF102CU, Package_SO:SOIC-8_3.9x4.9mm_P1.27mm
- removed U16: 74LS32, Package_SO:SOIC-14_3.9x8.7mm_P1.27mm
- removed U19, U21: NE555D, Package_SO:SOIC-8_3.9x4.9mm_P1.27mm
- added C1001: 100pF 50V, Capacitor_SMD:C_0603_1608Metric, F.Cu at (138.6, 134.2)
- added C1002: 100pF 50V, Capacitor_SMD:C_0603_1608Metric, F.Cu at (138.6, 136.7)
- added C1003: 100pF 50V, Capacitor_SMD:C_0603_1608Metric, F.Cu at (138.6, 139.2)
- added C1004: 100pF 50V, Capacitor_SMD:C_0603_1608Metric, F.Cu at (138.6, 141.7)
- added C1005: 100nF 100V, Capacitor_SMD:C_0603_1608Metric, F.Cu at (142.6, 134.2)
- added C1006: 100nF 100V, Capacitor_SMD:C_0603_1608Metric, F.Cu at (142.6, 136.7)
- added C1007: 100pF 50V, Capacitor_SMD:C_0603_1608Metric, F.Cu at (142.6, 139.2)
- added C1008: 100pF 50V, Capacitor_SMD:C_0603_1608Metric, F.Cu at (142.6, 141.7)
- added C1009: 100nF 100V, Capacitor_SMD:C_0603_1608Metric, F.Cu at (146.6, 134.2)
- added C1010: 10nF, Capacitor_SMD:C_0603_1608Metric_Pad1.08x0.95mm_HandSolder, F.Cu at (143.8, 114.0)
- added C1011: 100nF 100V, Capacitor_SMD:C_0603_1608Metric, F.Cu at (146.6, 136.7)
- added C1012: 10nF, Capacitor_SMD:C_0603_1608Metric_Pad1.08x0.95mm_HandSolder, F.Cu at (143.8, 116.5)
- added C1013: 100nF 100V, Capacitor_SMD:C_0603_1608Metric, F.Cu at (146.6, 139.2)
- added C1014: 100nF 100V, Capacitor_SMD:C_0603_1608Metric, F.Cu at (146.6, 141.7)
- added C201: 100nF 100V, Capacitor_SMD:C_0603_1608Metric, F.Cu at (104.0, 78.9)
- added C202: 100nF 100V, Capacitor_SMD:C_0603_1608Metric, F.Cu at (104.0, 81.4)
- added C203: 10uF 5%, Capacitor_SMD:C_0603_1608Metric, F.Cu at (104.0, 83.9)
- added C204: 100nF 100V, Capacitor_SMD:C_0603_1608Metric, F.Cu at (104.0, 86.5)
- added C205: 100nF 100V, Capacitor_SMD:C_0603_1608Metric, F.Cu at (104.0, 89.0)
- added C206: 100nF 100V, Capacitor_SMD:C_0603_1608Metric, F.Cu at (104.0, 91.5)
- added C207: 100nF 100V, Capacitor_SMD:C_0603_1608Metric, F.Cu at (104.0, 94.0)
- added C208: 100nF 100V, Capacitor_SMD:C_0603_1608Metric, F.Cu at (104.0, 96.5)
- added C209: 100nF 100V, Capacitor_SMD:C_0603_1608Metric, F.Cu at (104.0, 99.0)
- added C301: 27uF 5%, Capacitor_SMD:C_0603_1608Metric, F.Cu at (109.0, 34.8)
- added C302: 27uF 5%, Capacitor_SMD:C_0603_1608Metric, F.Cu at (109.0, 37.4)
- added C303: 10uF 5%, Capacitor_SMD:C_0603_1608Metric, F.Cu at (109.0, 39.9)
- added C304: 100nF 100V, Capacitor_SMD:C_0603_1608Metric, F.Cu at (109.0, 42.4)
- added C305: 100nF 100V, Capacitor_SMD:C_0603_1608Metric, F.Cu at (109.0, 44.9)
- added C306: 100nF 100V, Capacitor_SMD:C_0603_1608Metric, F.Cu at (113.0, 34.8)
- added C307: 100nF 100V, Capacitor_SMD:C_0603_1608Metric, F.Cu at (113.0, 37.4)
- added C308: 100nF 100V, Capacitor_SMD:C_0603_1608Metric, F.Cu at (113.0, 39.9)
- added C309: 100nF 100V, Capacitor_SMD:C_0603_1608Metric, F.Cu at (113.0, 42.4)
- added C310: 100nF 100V, Capacitor_SMD:C_0603_1608Metric, F.Cu at (113.0, 44.9)
- added C311: 100nF 100V, Capacitor_SMD:C_0603_1608Metric, F.Cu at (117.1, 34.8)
- added C312: 100nF 100V, Capacitor_SMD:C_0603_1608Metric, F.Cu at (117.1, 37.4)
- added C313: 100nF 100V, Capacitor_SMD:C_0603_1608Metric, F.Cu at (117.1, 39.9)
- added C401: 100nF 100V, Capacitor_SMD:C_0603_1608Metric, F.Cu at (77.5, 118.7)
- added C402: 100nF 100V, Capacitor_SMD:C_0603_1608Metric, F.Cu at (77.5, 121.2)
- added C403: 100nF 100V, Capacitor_SMD:C_0603_1608Metric, F.Cu at (77.5, 123.7)
- added C404: 100nF 100V, Capacitor_SMD:C_0603_1608Metric, F.Cu at (77.5, 126.3)
- added C405: 100nF 100V, Capacitor_SMD:C_0603_1608Metric, F.Cu at (77.5, 128.8)
- added C406: 470pF 50V, Capacitor_SMD:C_0603_1608Metric, F.Cu at (77.5, 131.3)
- added C407: 470pF 50V, Capacitor_SMD:C_0603_1608Metric, F.Cu at (77.5, 133.8)
- added C408: 100nF 100V, Capacitor_SMD:C_0603_1608Metric, F.Cu at (77.5, 136.3)
- added C701: 100nF 100V, Capacitor_SMD:C_0603_1608Metric, F.Cu at (117.1, 78.9)
- added C702: 100nF 100V, Capacitor_SMD:C_0603_1608Metric, F.Cu at (117.1, 81.4)
- added C703: 100nF 100V, Capacitor_SMD:C_0603_1608Metric, F.Cu at (117.1, 83.9)
- added C704: 100nF 100V, Capacitor_SMD:C_0603_1608Metric, F.Cu at (117.1, 86.5)
- added C705: 100nF 100V, Capacitor_SMD:C_0603_1608Metric, F.Cu at (117.1, 89.0)
- added C706: 100nF 100V, Capacitor_SMD:C_0603_1608Metric, F.Cu at (117.1, 91.5)
- added C707: 100nF 100V, Capacitor_SMD:C_0603_1608Metric, F.Cu at (121.1, 78.9)
- added C708: 100nF 100V, Capacitor_SMD:C_0603_1608Metric, F.Cu at (121.1, 81.4)
- added C710: 100nF 100V, Capacitor_SMD:C_0603_1608Metric, F.Cu at (121.1, 83.9)
- added C711: 100nF 100V, Capacitor_SMD:C_0603_1608Metric, F.Cu at (121.1, 86.5)
- added C712: 100pF, Capacitor_SMD:C_0603_1608Metric, F.Cu at (121.1, 89.0)
- added C901: 1uF, Capacitor_SMD:C_0603_1608Metric, F.Cu at (147.6, 61.5)
- added C902: 10uF, Capacitor_SMD:C_0603_1608Metric, F.Cu at (147.6, 64.0)
- added C903: 10uF, Capacitor_SMD:C_0603_1608Metric, F.Cu at (147.6, 66.6)
- added C904: 10uF, Capacitor_SMD:C_0603_1608Metric, F.Cu at (147.6, 69.1)
- added C905: 10uF, Capacitor_SMD:C_0603_1608Metric, F.Cu at (147.6, 71.6)
- added C906: 10uF, Capacitor_SMD:C_0603_1608Metric, F.Cu at (147.6, 74.1)
- added C907: 22uF, Capacitor_SMD:C_0603_1608Metric, F.Cu at (151.6, 61.5)
- added C908: 100nF 100V, Capacitor_SMD:C_0603_1608Metric, F.Cu at (151.6, 64.0)
- added C909: 100nF 100V, Capacitor_SMD:C_0603_1608Metric, F.Cu at (151.6, 66.6)
- added C913: 100nF 100V, Capacitor_SMD:C_0603_1608Metric, F.Cu at (151.6, 69.1)
- added C914: 100nF 100V, Capacitor_SMD:C_0603_1608Metric, F.Cu at (151.6, 71.6)
- added D1001: 1N4148W, Diode_SMD:D_SOD-123, F.Cu at (118.0, 140.8)
- added D1002: 1N4148W, Diode_SMD:D_SOD-123, F.Cu at (118.0, 144.2)
- added D701: MMBD914LT3G, Package_TO_SOT_SMD:SOT-23-3, F.Cu at (134.2, 103.9)
- added D702: MMBD914LT3G, Package_TO_SOT_SMD:SOT-23-3, F.Cu at (134.2, 108.4)
- added D703: RED [XL-2012SURC], LED_SMD:LED_0805_2012Metric_Pad1.15x1.40mm_HandSolder, F.Cu at (149.0, 79.2)
- added D704: GREEN [XL-2012UGC], LED_SMD:LED_0805_2012Metric_Pad1.15x1.40mm_HandSolder, F.Cu at (149.0, 82.2)
- added D901: RED [XL-2012SURC], LED_SMD:LED_0805_2012Metric_Pad1.15x1.40mm_HandSolder, F.Cu at (138.7, 59.7)
- added D902: RED [XL-2012SURC], LED_SMD:LED_0805_2012Metric_Pad1.15x1.40mm_HandSolder, F.Cu at (138.7, 62.7)
- added D903: RED [XL-2012SURC], LED_SMD:LED_0805_2012Metric_Pad1.15x1.40mm_HandSolder, F.Cu at (138.7, 65.7)
- added D904: GREEN [XL-2012UGC], LED_SMD:LED_0805_2012Metric_Pad1.15x1.40mm_HandSolder, F.Cu at (138.7, 68.8)
- added D905: 1N5819WS, Diode_SMD:D_SOD-323, F.Cu at (157.7, 35.1)
- added D907: GREEN [XL-2012UGC], LED_SMD:LED_0805_2012Metric_Pad1.15x1.40mm_HandSolder, F.Cu at (138.7, 71.8)
- added J1001: Conn_02x02_Odd_Even, Connector_PinHeader_2.54mm:PinHeader_2x02_P2.54mm_Vertical, F.Cu at (130.5, 141.4)
- added J201: Conn_02x02_Odd_Even, Connector_PinHeader_2.54mm:PinHeader_2x02_P2.54mm_Vertical, F.Cu at (108.3, 89.6)
- added J202: Conn_02x03_Odd_Even, Connector_PinHeader_2.54mm:PinHeader_2x03_P2.54mm_Vertical, F.Cu at (108.3, 80.0)
- added J203: Conn_01x02, Connector_PinHeader_1.27mm:PinHeader_1x02_P1.27mm_Vertical, F.Cu at (108.1, 96.1)
- added J301: Conn_02x03_Odd_Even, Connector_PinHeader_2.54mm:PinHeader_2x03_P2.54mm_Vertical, F.Cu at (112.3, 68.3)
- added J303: Conn_01x02, Connector_PinHeader_1.27mm:PinHeader_1x02_P1.27mm_Vertical, F.Cu at (109.1, 47.8)
- added J304: Conn_02x04_Odd_Even, Connector_PinHeader_2.54mm:PinHeader_2x04_P2.54mm_Vertical, F.Cu at (112.3, 56.1)
- added J401: Conn_01x02, Jumper:SolderJumper-2_P1.3mm_Open_TrianglePad1.0x1.5mm, F.Cu at (81.6, 136.8)
- added J402: Conn_01x02, Jumper:SolderJumper-2_P1.3mm_Open_TrianglePad1.0x1.5mm, F.Cu at (81.6, 140.4)
- added J701: Conn_02x02_Odd_Even, Connector_PinHeader_2.54mm:PinHeader_2x02_P2.54mm_Vertical, F.Cu at (117.4, 95.0)
- added J702: Conn_02x02_Odd_Even, Connector_PinHeader_2.54mm:PinHeader_2x02_P2.54mm_Vertical, F.Cu at (117.4, 102.2)
- added J801: Conn_02x03_Odd_Even, Connector_PinHeader_2.54mm:PinHeader_2x03_P2.54mm_Vertical, F.Cu at (156.1, 80.0)
- added J902: 54-00164, 54-00164:TENSILITY_54-00164, F.Cu at (129.0, 66.4)
- added J904: USB-B-S-X-X-VT, USB_B_S_VT:USB-B-S-VT, F.Cu at (165.4, 104.2)
- added J905: Conn_01x06, Connector_PinHeader_2.54mm:PinHeader_1x06_P2.54mm_Vertical, F.Cu at (147.9, 45.3)
- added R1001: 1KΩ, Resistor_SMD:R_0603_1608Metric_Pad0.98x0.95mm_HandSolder, F.Cu at (143.8, 119.0)
- added R1002: 51KΩ, Resistor_SMD:R_0603_1608Metric_Pad0.98x0.95mm_HandSolder, F.Cu at (143.8, 121.5)
- added R1003: PV36W104C01B00, PV36W104C01B00:POT_PV36W_BRN, F.Cu at (120.0, 116.0)
- added R1004: 10KΩ, Resistor_SMD:R_0603_1608Metric_Pad0.98x0.95mm_HandSolder, F.Cu at (143.8, 124.0)
- added R1005: 10KΩ, Resistor_SMD:R_0603_1608Metric_Pad0.98x0.95mm_HandSolder, F.Cu at (143.8, 126.5)
- added R1006: 100KΩ, Resistor_SMD:R_0603_1608Metric_Pad0.98x0.95mm_HandSolder, F.Cu at (148.2, 114.0)
- added R1007: PV36W204C01B00, PV36W104C01B00:POT_PV36W_BRN, F.Cu at (120.0, 122.6)
- added R1008: PV36W104C01B00, PV36W104C01B00:POT_PV36W_BRN, F.Cu at (120.0, 129.2)
- added R1009: 10KΩ, Resistor_SMD:R_0603_1608Metric_Pad0.98x0.95mm_HandSolder, F.Cu at (148.2, 116.5)
- added R1010: 1MΩ 5%, Resistor_SMD:R_0603_1608Metric_Pad0.98x0.95mm_HandSolder, F.Cu at (148.2, 119.0)
- added R1011: 680Ω, Resistor_SMD:R_0603_1608Metric_Pad0.98x0.95mm_HandSolder, F.Cu at (148.2, 121.5)
- added R1012: PV36W103C01B00, PV36W104C01B00:POT_PV36W_BRN, F.Cu at (120.0, 135.8)
- added R1013: 1KΩ, Resistor_SMD:R_0603_1608Metric_Pad0.98x0.95mm_HandSolder, F.Cu at (148.2, 124.0)
- added R201: PV36W104C01B00, PV36W104C01B00:POT_PV36W_BRN, F.Cu at (80.4, 80.9)
- added R202: 10K, Resistor_SMD:R_0603_1608Metric_Pad0.98x0.95mm_HandSolder, F.Cu at (99.1, 104.2)
- added R203: PV36W104C01B00, PV36W104C01B00:POT_PV36W_BRN, F.Cu at (80.4, 87.5)
- added R204: PV36W104C01B00, PV36W104C01B00:POT_PV36W_BRN, F.Cu at (80.4, 94.1)
- added R205: 1MΩ 5%, Resistor_SMD:R_0603_1608Metric_Pad0.98x0.95mm_HandSolder, F.Cu at (99.1, 106.7)
- added R206: 10KΩ, Resistor_SMD:R_0603_1608Metric_Pad0.98x0.95mm_HandSolder, F.Cu at (99.1, 109.2)
- added R207: 10KΩ, Resistor_SMD:R_0603_1608Metric_Pad0.98x0.95mm_HandSolder, F.Cu at (99.1, 111.7)
- added R208: PV36W204C01B00, PV36W104C01B00:POT_PV36W_BRN, F.Cu at (80.4, 100.8)
- added R209: 10kΩ, Resistor_SMD:R_0603_1608Metric_Pad0.98x0.95mm_HandSolder, F.Cu at (99.1, 114.2)
- added R210: 10K, Resistor_SMD:R_0603_1608Metric_Pad0.98x0.95mm_HandSolder, F.Cu at (103.5, 104.2)
- added R211: 10kΩ, Resistor_SMD:R_0603_1608Metric_Pad0.98x0.95mm_HandSolder, F.Cu at (103.5, 106.7)
- added R212: PV36W104C01B00, PV36W104C01B00:POT_PV36W_BRN, F.Cu at (80.4, 107.4)
- added R213: 10kΩ, Resistor_SMD:R_0603_1608Metric_Pad0.98x0.95mm_HandSolder, F.Cu at (103.5, 109.2)
- added R214: 10K, Resistor_SMD:R_0603_1608Metric_Pad0.98x0.95mm_HandSolder, F.Cu at (103.5, 111.7)
- added R215: 10K, Resistor_SMD:R_0603_1608Metric_Pad0.98x0.95mm_HandSolder, F.Cu at (103.5, 114.2)
- added R216: 10kΩ, Resistor_SMD:R_0603_1608Metric_Pad0.98x0.95mm_HandSolder, F.Cu at (107.8, 104.2)
- added R217: 10kΩ, Resistor_SMD:R_0603_1608Metric_Pad0.98x0.95mm_HandSolder, F.Cu at (107.8, 106.7)
- added R218: 10kΩ, Resistor_SMD:R_0603_1608Metric_Pad0.98x0.95mm_HandSolder, F.Cu at (107.8, 109.2)
- added R219: 10kΩ, Resistor_SMD:R_0603_1608Metric_Pad0.98x0.95mm_HandSolder, F.Cu at (107.8, 111.7)
- added R220: 10kΩ, Resistor_SMD:R_0603_1608Metric_Pad0.98x0.95mm_HandSolder, F.Cu at (107.8, 114.2)
- added R301: PV36W104C01B00, PV36W104C01B00:POT_PV36W_BRN, F.Cu at (80.4, 36.8)
- added R302: 10K, Resistor_SMD:R_0603_1608Metric_Pad0.98x0.95mm_HandSolder, F.Cu at (99.1, 55.0)
- added R303: PV36W104C01B00, PV36W104C01B00:POT_PV36W_BRN, F.Cu at (80.4, 43.4)
- added R304: 301kΩ 1%, Resistor_SMD:R_0603_1608Metric_Pad0.98x0.95mm_HandSolder, F.Cu at (99.1, 57.6)
- added R305: 10.2kΩ 1%, Resistor_SMD:R_0603_1608Metric_Pad0.98x0.95mm_HandSolder, F.Cu at (99.1, 60.1)
- added R306: PV36W104C01B00, PV36W104C01B00:POT_PV36W_BRN, F.Cu at (80.4, 50.1)
- added R307: 10kΩ, Resistor_SMD:R_0603_1608Metric_Pad0.98x0.95mm_HandSolder, F.Cu at (99.1, 62.6)
- added R308: 10K, Resistor_SMD:R_0603_1608Metric_Pad0.98x0.95mm_HandSolder, F.Cu at (99.1, 65.1)
- added R309: 10K, Resistor_SMD:R_0603_1608Metric_Pad0.98x0.95mm_HandSolder, F.Cu at (99.1, 67.6)
- added R310: 10K, Resistor_SMD:R_0603_1608Metric_Pad0.98x0.95mm_HandSolder, F.Cu at (99.1, 70.1)
- added R311: 976kΩ 1%, Resistor_SMD:R_0603_1608Metric_Pad0.98x0.95mm_HandSolder, F.Cu at (99.1, 72.6)
- added R312: 1MΩ 5%, Resistor_SMD:R_0603_1608Metric_Pad0.98x0.95mm_HandSolder, F.Cu at (103.5, 55.0)
- added R313: 10kΩ, Resistor_SMD:R_0603_1608Metric_Pad0.98x0.95mm_HandSolder, F.Cu at (103.5, 57.6)
- added R314: 402kΩ 1%, Resistor_SMD:R_0603_1608Metric_Pad0.98x0.95mm_HandSolder, F.Cu at (103.5, 60.1)
- added R315: 6.65kΩ 1%, Resistor_SMD:R_0603_1608Metric_Pad0.98x0.95mm_HandSolder, F.Cu at (103.5, 62.6)
- added R316: 10kΩ, Resistor_SMD:R_0603_1608Metric_Pad0.98x0.95mm_HandSolder, F.Cu at (103.5, 65.1)
- added R317: 10KΩ, Resistor_SMD:R_0603_1608Metric_Pad0.98x0.95mm_HandSolder, F.Cu at (103.5, 67.6)
- added R318: 10kΩ 1%, Resistor_SMD:R_0603_1608Metric_Pad0.98x0.95mm_HandSolder, F.Cu at (103.5, 70.1)
- added R319: 10kΩ, Resistor_SMD:R_0603_1608Metric_Pad0.98x0.95mm_HandSolder, F.Cu at (103.5, 72.6)
- added R320: PV36W104C01B00, PV36W104C01B00:POT_PV36W_BRN, F.Cu at (80.4, 56.7)
- added R321: PV36W204C01B00, PV36W104C01B00:POT_PV36W_BRN, F.Cu at (80.4, 63.3)
- added R322: 10kΩ, Resistor_SMD:R_0603_1608Metric_Pad0.98x0.95mm_HandSolder, F.Cu at (107.8, 55.0)
- added R323: 10kΩ, Resistor_SMD:R_0603_1608Metric_Pad0.98x0.95mm_HandSolder, F.Cu at (107.8, 57.6)
- added R324: 10K, Resistor_SMD:R_0603_1608Metric_Pad0.98x0.95mm_HandSolder, F.Cu at (107.8, 60.1)
- added R325: 10K, Resistor_SMD:R_0603_1608Metric_Pad0.98x0.95mm_HandSolder, F.Cu at (107.8, 62.6)
- added R326: 10kΩ, Resistor_SMD:R_0603_1608Metric_Pad0.98x0.95mm_HandSolder, F.Cu at (107.8, 65.1)
- added R327: PV36W104C01B00, PV36W104C01B00:POT_PV36W_BRN, F.Cu at (80.4, 69.9)
- added R328: 10kΩ, Resistor_SMD:R_0603_1608Metric_Pad0.98x0.95mm_HandSolder, F.Cu at (107.8, 67.6)
- added R329: 10kΩ, Resistor_SMD:R_0603_1608Metric_Pad0.98x0.95mm_HandSolder, F.Cu at (107.8, 70.1)
- added R401: 1KΩ, Resistor_SMD:R_0603_1608Metric_Pad0.98x0.95mm_HandSolder, F.Cu at (81.6, 118.7)
- added R402: 1KΩ, Resistor_SMD:R_0603_1608Metric_Pad0.98x0.95mm_HandSolder, F.Cu at (81.6, 121.2)
- added R403: 1KΩ, Resistor_SMD:R_0603_1608Metric_Pad0.98x0.95mm_HandSolder, F.Cu at (81.6, 123.7)
- added R404: PV36W502C01B00, PV36W104C01B00:POT_PV36W_BRN, F.Cu at (88.7, 120.7)
- added R405: PV36W502C01B00, PV36W104C01B00:POT_PV36W_BRN, F.Cu at (88.7, 127.3)
- added R406: 500Ω, Resistor_SMD:R_0603_1608Metric_Pad0.98x0.95mm_HandSolder, F.Cu at (81.6, 126.3)
- added R407: 500Ω, Resistor_SMD:R_0603_1608Metric_Pad0.98x0.95mm_HandSolder, F.Cu at (81.6, 128.8)
- added R408: 100KΩ, Resistor_SMD:R_0603_1608Metric_Pad0.98x0.95mm_HandSolder, F.Cu at (81.6, 131.3)
- added R409: 100KΩ, Resistor_SMD:R_0603_1608Metric_Pad0.98x0.95mm_HandSolder, F.Cu at (81.6, 133.8)
- added R701: PV36W104C01B00, PV36W104C01B00:POT_PV36W_BRN, F.Cu at (141.7, 104.9)
- added R702: 10KΩ, Resistor_SMD:R_0603_1608Metric_Pad0.98x0.95mm_HandSolder, F.Cu at (135.7, 78.9)
- added R703: 10KΩ, Resistor_SMD:R_0603_1608Metric_Pad0.98x0.95mm_HandSolder, F.Cu at (135.7, 81.4)
- added R704: 10KΩ, Resistor_SMD:R_0603_1608Metric_Pad0.98x0.95mm_HandSolder, F.Cu at (135.7, 83.9)
- added R705: 10KΩ, Resistor_SMD:R_0603_1608Metric_Pad0.98x0.95mm_HandSolder, F.Cu at (135.7, 86.5)
- added R706: 10KΩ, Resistor_SMD:R_0603_1608Metric_Pad0.98x0.95mm_HandSolder, F.Cu at (135.7, 89.0)
- added R707: 10KΩ, Resistor_SMD:R_0603_1608Metric_Pad0.98x0.95mm_HandSolder, F.Cu at (140.0, 78.9)
- added R708: 10KΩ, Resistor_SMD:R_0603_1608Metric_Pad0.98x0.95mm_HandSolder, F.Cu at (140.0, 81.4)
- added R709: 1KΩ, Resistor_SMD:R_0603_1608Metric_Pad0.98x0.95mm_HandSolder, F.Cu at (140.0, 83.9)
- added R710: 1KΩ, Resistor_SMD:R_0603_1608Metric_Pad0.98x0.95mm_HandSolder, F.Cu at (140.0, 86.5)
- added R711: 100Ω, Resistor_SMD:R_0603_1608Metric_Pad0.98x0.95mm_HandSolder, F.Cu at (140.0, 89.0)
- added R712: 1KΩ, Resistor_SMD:R_0603_1608Metric_Pad0.98x0.95mm_HandSolder, F.Cu at (144.4, 78.9)
- added R713: 1KΩ, Resistor_SMD:R_0603_1608Metric_Pad0.98x0.95mm_HandSolder, F.Cu at (144.4, 81.4)
- added R714: 470Ω, Resistor_SMD:R_0603_1608Metric_Pad0.98x0.95mm_HandSolder, F.Cu at (144.4, 83.9)
- added R715: 470Ω, Resistor_SMD:R_0603_1608Metric_Pad0.98x0.95mm_HandSolder, F.Cu at (144.4, 86.5)
- added R901: 10KΩ, Resistor_SMD:R_0603_1608Metric_Pad0.98x0.95mm_HandSolder, F.Cu at (143.4, 44.2)
- added R902: 10KΩ, Resistor_SMD:R_0603_1608Metric_Pad0.98x0.95mm_HandSolder, F.Cu at (143.4, 46.8)
- added R903: PV36W104C01B00, PV36W104C01B00:POT_PV36W_BRN, F.Cu at (147.4, 36.8)
- added R906: 470Ω, Resistor_SMD:R_0603_1608Metric_Pad0.98x0.95mm_HandSolder, F.Cu at (143.4, 49.3)
- added R907: 470Ω, Resistor_SMD:R_0603_1608Metric_Pad0.98x0.95mm_HandSolder, F.Cu at (143.4, 51.8)
- added R908: 470Ω, Resistor_SMD:R_0603_1608Metric_Pad0.98x0.95mm_HandSolder, F.Cu at (143.4, 54.3)
- added R909: 470Ω, Resistor_SMD:R_0603_1608Metric_Pad0.98x0.95mm_HandSolder, F.Cu at (143.4, 56.8)
- added R911: 10Ω, Resistor_SMD:R_0603_1608Metric_Pad0.98x0.95mm_HandSolder, F.Cu at (143.4, 59.3)
- added TP1001: TestPoint, TestPoint:TestPoint_Loop_D2.60mm_Drill1.6mm_Beaded, F.Cu at (139.1, 115.2)
- added TP1002: TestPoint, TestPoint:TestPoint_Loop_D2.60mm_Drill1.6mm_Beaded, F.Cu at (139.1, 120.3)
- added TP1003: TestPoint, TestPoint:TestPoint_Loop_D2.60mm_Drill1.6mm_Beaded, F.Cu at (139.1, 125.3)
- added TP1004: TestPoint, TestPoint:TestPoint_Loop_D2.60mm_Drill1.6mm_Beaded, F.Cu at (139.1, 130.4)
- added TP201: TestPoint, TestPoint:TestPoint_Loop_D2.60mm_Drill1.6mm_Beaded, F.Cu at (99.5, 80.2)
- added TP202: TestPoint, TestPoint:TestPoint_Loop_D2.60mm_Drill1.6mm_Beaded, F.Cu at (99.5, 85.2)
- added TP203: TestPoint, TestPoint:TestPoint_Loop_D2.60mm_Drill1.6mm_Beaded, F.Cu at (99.5, 90.3)
- added TP204: TestPoint, TestPoint:TestPoint_Loop_D2.60mm_Drill1.6mm_Beaded, F.Cu at (99.5, 95.3)
- added TP205: TestPoint, TestPoint:TestPoint_Loop_D2.60mm_Drill1.6mm_Beaded, F.Cu at (99.5, 100.4)
- added TP301: TestPoint, TestPoint:TestPoint_Loop_D2.60mm_Drill1.6mm_Beaded, F.Cu at (99.5, 36.1)
- added TP302: TestPoint, TestPoint:TestPoint_Loop_D2.60mm_Drill1.6mm_Beaded, F.Cu at (99.5, 41.2)
- added TP303: TestPoint, TestPoint:TestPoint_Loop_D2.60mm_Drill1.6mm_Beaded, F.Cu at (99.5, 46.2)
- added TP304: TestPoint, TestPoint:TestPoint_Loop_D2.60mm_Drill1.6mm_Beaded, F.Cu at (99.5, 51.3)
- added TP305: TestPoint, TestPoint:TestPoint_Loop_D2.60mm_Drill1.6mm_Beaded, F.Cu at (104.5, 36.1)
- added TP306: TestPoint, TestPoint:TestPoint_Loop_D2.60mm_Drill1.6mm_Beaded, F.Cu at (104.5, 41.2)
- added TP307: TestPoint, TestPoint:TestPoint_Loop_D2.60mm_Drill1.6mm_Beaded, F.Cu at (104.5, 46.2)
- added TP401: TestPoint, TestPoint:TestPoint_Loop_D2.60mm_Drill1.6mm_Beaded, F.Cu at (100.4, 139.8)
- added TP701: TestPoint, TestPoint:TestPoint_Loop_D2.60mm_Drill1.6mm_Beaded, F.Cu at (134.1, 94.1)
- added TP702: TestPoint, TestPoint:TestPoint_Loop_D2.60mm_Drill1.6mm_Beaded, F.Cu at (134.1, 99.2)
- added TP703: TestPoint, TestPoint:TestPoint_Loop_D2.60mm_Drill1.6mm_Beaded, F.Cu at (139.2, 94.1)
- added TP704: TestPoint, TestPoint:TestPoint_Loop_D2.60mm_Drill1.6mm_Beaded, F.Cu at (139.2, 99.2)
- added TP705: TestPoint, TestPoint:TestPoint_Loop_D2.60mm_Drill1.6mm_Beaded, F.Cu at (144.2, 94.1)
- added TP706: TestPoint, TestPoint:TestPoint_Loop_D2.60mm_Drill1.6mm_Beaded, F.Cu at (144.2, 99.2)
- added TP707: TestPoint, TestPoint:TestPoint_Loop_D2.60mm_Drill1.6mm_Beaded, F.Cu at (149.3, 94.1)
- added TP708: TestPoint, TestPoint:TestPoint_Loop_D2.60mm_Drill1.6mm_Beaded, F.Cu at (149.3, 99.2)
- added TP901: TestPoint, TestPoint:TestPoint_Loop_D2.60mm_Drill1.6mm_Beaded, F.Cu at (123.6, 45.5)
- added TP902: TestPoint, TestPoint:TestPoint_Loop_D2.60mm_Drill1.6mm_Beaded, F.Cu at (123.6, 50.6)
- added TP904: TestPoint, TestPoint:TestPoint_Loop_D2.60mm_Drill1.6mm_Beaded, F.Cu at (123.6, 55.6)
- added TP905: TestPoint, TestPoint:TestPoint_Loop_D2.60mm_Drill1.6mm_Beaded, F.Cu at (128.6, 45.5)
- added TP906: TestPoint, TestPoint:TestPoint_Loop_D2.60mm_Drill1.6mm_Beaded, F.Cu at (128.6, 50.6)
- added TP907: TestPoint, TestPoint:TestPoint_Loop_D2.60mm_Drill1.6mm_Beaded, F.Cu at (128.6, 55.6)
- added TP908: TestPoint, TestPoint:TestPoint_Loop_D2.60mm_Drill1.6mm_Beaded, F.Cu at (133.7, 45.5)
- added TP909: TestPoint, TestPoint:TestPoint_Loop_D2.60mm_Drill1.6mm_Beaded, F.Cu at (133.7, 50.6)
- added TP910: TestPoint, TestPoint:TestPoint_Loop_D2.60mm_Drill1.6mm_Beaded, F.Cu at (133.7, 55.6)
- added TP911: TestPoint, TestPoint:TestPoint_Loop_D2.60mm_Drill1.6mm_Beaded, F.Cu at (138.7, 45.5)
- added TP912: TestPoint, TestPoint:TestPoint_Loop_D2.60mm_Drill1.6mm_Beaded, F.Cu at (138.7, 50.6)
- added TP913: TestPoint, TestPoint:TestPoint_Loop_D2.60mm_Drill1.6mm_Beaded, F.Cu at (138.7, 55.6)
- added U1001: NE555D, Package_SO:SOIC-8_3.9x4.9mm_P1.27mm, F.Cu at (132.4, 116.1)
- added U1002: NE555D, Package_SO:SOIC-8_3.9x4.9mm_P1.27mm, F.Cu at (132.4, 122.7)
- added U1003: TL082, Package_SO:SOIC-8_3.9x4.9mm_P1.27mm, F.Cu at (132.4, 129.2)
- added U1004: TL082, Package_SO:SOIC-8_3.9x4.9mm_P1.27mm, F.Cu at (132.4, 135.8)
- added U201: TL082, Package_SO:SOIC-8_3.9x4.9mm_P1.27mm, F.Cu at (92.7, 81.0)
- added U202: TL082, Package_SO:SOIC-8_3.9x4.9mm_P1.27mm, F.Cu at (92.7, 87.6)
- added U203: TL082, Package_SO:SOIC-8_3.9x4.9mm_P1.27mm, F.Cu at (92.7, 94.2)
- added U204: TL082, Package_SO:SOIC-8_3.9x4.9mm_P1.27mm, F.Cu at (92.7, 100.8)
- added U301: TL082, Package_SO:SOIC-8_3.9x4.9mm_P1.27mm, F.Cu at (92.7, 37.0)
- added U302: TL082, Package_SO:SOIC-8_3.9x4.9mm_P1.27mm, F.Cu at (92.7, 43.5)
- added U303: TL082, Package_SO:SOIC-8_3.9x4.9mm_P1.27mm, F.Cu at (92.7, 50.1)
- added U304: TL082, Package_SO:SOIC-8_3.9x4.9mm_P1.27mm, F.Cu at (92.7, 56.7)
- added U305: TL082, Package_SO:SOIC-8_3.9x4.9mm_P1.27mm, F.Cu at (92.7, 63.3)
- added U401: LM311, Package_SO:SOIC-8_3.9x4.9mm_P1.27mm, F.Cu at (96.5, 134.1)
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
Commit message: commits latest kiCAD project for BOM generation
Parts:
- removed C901: 1uF, Capacitor_SMD:C_0603_1608Metric
- removed C902, C903, C904, C905, C906: 10uF, Capacitor_SMD:C_0603_1608Metric
- removed C907: 22uF, Capacitor_SMD:C_0603_1608Metric
- removed C908, C909, C913, C914: 100nF 100V, Capacitor_SMD:C_0603_1608Metric
- removed D901, D902, D903: RED [XL-2012SURC], LED_SMD:LED_0805_2012Metric_Pad1.15x1.40mm_HandSolder
- removed D904, D907: GREEN [XL-2012UGC], LED_SMD:LED_0805_2012Metric_Pad1.15x1.40mm_HandSolder
- removed D905: 1N5819WS, Diode_SMD:D_SOD-323
- removed J902: 54-00164, 54-00164:TENSILITY_54-00164
- removed J904: USB-B-S-X-X-VT, USB_B_S_VT:USB-B-S-VT
- removed J905: Conn_01x06, Connector_PinHeader_2.54mm:PinHeader_1x06_P2.54mm_Vertical
- removed R901, R902: 10KΩ, Resistor_SMD:R_0603_1608Metric_Pad0.98x0.95mm_HandSolder
- removed R903: PV36W104C01B00, PV36W104C01B00:POT_PV36W_BRN
- removed R906, R907, R908, R909: 470Ω, Resistor_SMD:R_0603_1608Metric_Pad0.98x0.95mm_HandSolder
- removed R911: 10Ω, Resistor_SMD:R_0603_1608Metric_Pad0.98x0.95mm_HandSolder
- removed TP901, TP902, TP904, TP905, TP906, TP907, TP908, TP909, TP910, TP911, TP912, TP913: TestPoint, TestPoint:TestPoint_Loop_D2.60mm_Drill1.6mm_Beaded
- removed U901: REF102CU, Package_SO:SOIC-8_3.9x4.9mm_P1.27mm
- removed U902, U903: TL082, Package_SO:SOIC-8_3.9x4.9mm_P1.27mm
- removed U904: AMS1117-3.3, Package_TO_SOT_SMD:SOT-223-3_TabPin2
- removed U905: TMH 0515D, TMH_0515D:TMH DUAL_TRP
- removed U906: R-78E5.0-0.5, R_78E5_0_0_5:R_78E_0.5_RCP
- added C501: 10uF, Capacitor_SMD:C_0603_1608Metric, F.Cu at (186.5, 67.5)
- added C502: 1uF, Capacitor_SMD:C_0603_1608Metric, F.Cu at (186.5, 70.0)
- added C503: 100nF 100V, Capacitor_SMD:C_0603_1608Metric, F.Cu at (186.5, 72.5)
- added C504: 100nF 100V, Capacitor_SMD:C_0603_1608Metric, F.Cu at (186.5, 75.0)
- added C505: 10uF, Capacitor_SMD:C_0603_1608Metric, F.Cu at (186.5, 77.5)
- added C506: 100nF 100V, Capacitor_SMD:C_0603_1608Metric, F.Cu at (186.5, 80.0)
- added C507: 100nF 100V, Capacitor_SMD:C_0603_1608Metric, F.Cu at (190.5, 67.5)
- added C508: 10uF, Capacitor_SMD:C_0603_1608Metric, F.Cu at (190.5, 70.0)
- added C509: 10uF, Capacitor_SMD:C_0603_1608Metric, F.Cu at (190.5, 72.5)
- added C510: 10uF, Capacitor_SMD:C_0603_1608Metric, F.Cu at (190.5, 75.0)
- added C511: 22uF, Capacitor_SMD:C_0603_1608Metric, F.Cu at (190.5, 77.5)
- added D501: GREEN [XL-2012UGC], LED_SMD:LED_0805_2012Metric_Pad1.15x1.40mm_HandSolder, F.Cu at (204.3, 48.0)
- added D502: GREEN [XL-2012UGC], LED_SMD:LED_0805_2012Metric_Pad1.15x1.40mm_HandSolder, F.Cu at (204.3, 51.0)
- added D503: RED [XL-2012SURC], LED_SMD:LED_0805_2012Metric_Pad1.15x1.40mm_HandSolder, F.Cu at (204.3, 54.1)
- added D504: RED [XL-2012SURC], LED_SMD:LED_0805_2012Metric_Pad1.15x1.40mm_HandSolder, F.Cu at (204.3, 57.1)
- added D505: RED [XL-2012SURC], LED_SMD:LED_0805_2012Metric_Pad1.15x1.40mm_HandSolder, F.Cu at (204.3, 60.2)
- added D506: 1N5819WS, Diode_SMD:D_SOD-323, F.Cu at (197.7, 38.6)
- added J501: 54-00164, 54-00164:TENSILITY_54-00164, F.Cu at (200.9, 72.3)
- added J502: 5227699-1, 5227699:TE_5227699-1, F.Cu at (214.4, 169.7)
- added J503: USB-B-S-X-X-VT, USB_B_S_VT:USB-B-S-VT, F.Cu at (421.9, 167.6)
- added J504: Conn_01x06, Connector_PinHeader_2.54mm:PinHeader_1x06_P2.54mm_Vertical, F.Cu at (199.6, 48.8)
- added R501: 500Ω, Resistor_SMD:R_0603_1608Metric_Pad0.98x0.95mm_HandSolder, F.Cu at (195.1, 47.7)
- added R502: 10KΩ, Resistor_SMD:R_0603_1608Metric_Pad0.98x0.95mm_HandSolder, F.Cu at (195.1, 50.2)
- added R503: 100Ω, Resistor_SMD:R_0603_1608Metric_Pad0.98x0.95mm_HandSolder, F.Cu at (195.1, 52.8)
- added R504: 10KΩ, Resistor_SMD:R_0603_1608Metric_Pad0.98x0.95mm_HandSolder, F.Cu at (195.1, 55.3)
- added R505: 330Ω, Resistor_SMD:R_0603_1608Metric_Pad0.98x0.95mm_HandSolder, F.Cu at (195.1, 57.8)
- added R506: PV36W104C01B00, PV36W104C01B00:POT_PV36W_BRN, F.Cu at (169.2, 75.0)
- added R507: 1KΩ, Resistor_SMD:R_0603_1608Metric_Pad0.98x0.95mm_HandSolder, F.Cu at (195.1, 60.3)
- added R508: 1KΩ, Resistor_SMD:R_0603_1608Metric_Pad0.98x0.95mm_HandSolder, F.Cu at (195.1, 62.8)
- added SW701: PTS636SL43SMTRLFS, PTS636SL43SMTRLFS:PTS636SL43SMTRLFS, F.Cu at (154.2, 135.7)
- added SW704: PTS636SL43SMTRLFS, PTS636SL43SMTRLFS:PTS636SL43SMTRLFS, F.Cu at (152.9, 126.8)
- added TP501: TestPoint, TestPoint:TestPoint_Loop_D2.60mm_Drill1.6mm_Beaded, F.Cu at (166.8, 49.0)
- added TP502: TestPoint, TestPoint:TestPoint_Loop_D2.60mm_Drill1.6mm_Beaded, F.Cu at (166.8, 54.1)
- added TP503: TestPoint, TestPoint:TestPoint_Loop_D2.60mm_Drill1.6mm_Beaded, F.Cu at (166.8, 59.1)
- added TP504: TestPoint, TestPoint:TestPoint_Loop_D2.60mm_Drill1.6mm_Beaded, F.Cu at (171.9, 49.0)
- added TP505: TestPoint, TestPoint:TestPoint_Loop_D2.60mm_Drill1.6mm_Beaded, F.Cu at (171.9, 54.1)
- added TP506: TestPoint, TestPoint:TestPoint_Loop_D2.60mm_Drill1.6mm_Beaded, F.Cu at (171.9, 59.1)
- added TP507: TestPoint, TestPoint:TestPoint_Loop_D2.60mm_Drill1.6mm_Beaded, F.Cu at (176.9, 49.0)
- added TP508: TestPoint, TestPoint:TestPoint_Loop_D2.60mm_Drill1.6mm_Beaded, F.Cu at (176.9, 54.1)
- added TP509: TestPoint, TestPoint:TestPoint_Loop_D2.60mm_Drill1.6mm_Beaded, F.Cu at (176.9, 59.1)
- added TP510: TestPoint, TestPoint:TestPoint_Loop_D2.60mm_Drill1.6mm_Beaded, F.Cu at (182.0, 49.0)
- added TP511: TestPoint, TestPoint:TestPoint_Loop_D2.60mm_Drill1.6mm_Beaded, F.Cu at (182.0, 54.1)
- added TP512: TestPoint, TestPoint:TestPoint_Loop_D2.60mm_Drill1.6mm_Beaded, F.Cu at (182.0, 59.1)
- added U501: REF102CU, Package_SO:SOIC-8_3.9x4.9mm_P1.27mm, F.Cu at (188.7, 49.8)
- added U502: R-78E5.0-0.5, R_78E5_0_0_5:R_78E_0.5_RCP, F.Cu at (168.4, 69.0)
- added U503: TL082, Package_SO:SOIC-8_3.9x4.9mm_P1.27mm, F.Cu at (188.7, 56.4)
- added U504: TL082, Package_SO:SOIC-8_3.9x4.9mm_P1.27mm, F.Cu at (188.7, 63.0)
- added U505: TMH 0515D, TMH_0515D:TMH DUAL_TRP, F.Cu at (167.3, 39.3)
- added U506: AMS1117-3.3, Package_TO_SOT_SMD:SOT-223-3_TabPin2, F.Cu at (190.6, 41.3)
- D701, D702: footprint Package_TO_SOT_SMD:SOT-23-3 -> MMBD914LT3G:SOT-23_ONS
- moved R301 296.2 mm to (320.9, 209.6)
- moved R320 291.1 mm to (321.1, 220.5)
- moved TP303 290.1 mm to (331.3, 220.5)
- moved R327 288.8 mm to (337.3, 201.7)
- moved U304 272.8 mm to (314.0, 216.2)
- moved C1006 271.0 mm to (376.8, 273.0)
- moved C1007 271.0 mm to (376.8, 275.5)
- moved C1008 271.0 mm to (376.8, 278.0)
- moved C1010 271.0 mm to (378.0, 250.3)
- moved C1011 271.0 mm to (380.8, 273.0)
- moved C1012 271.0 mm to (378.0, 252.8)
- moved C1013 271.0 mm to (380.8, 275.5)
- moved C1014 271.0 mm to (380.8, 278.0)
- moved D1001 271.0 mm to (352.3, 277.2)
- moved D1002 271.0 mm to (352.3, 280.5)
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Other:
- board outline added: 228.6 x 81 mm
