File: HB_Drive_V1/HB_Drive_V1.kicad_pcb (KiCad board)
At the start: 2 copper layers, 228.6 x 81 mm, 255 parts, among them J1001 Conn_02x02_Odd_Even, J201 Conn_02x02_Odd_Even, J202 Conn_02x03_Odd_Even, J203 Conn_01x02, J301 Conn_02x03_Odd_Even, J303 Conn_01x02, J304 Conn_02x04_Odd_Even, J401 Conn_01x02, J402 Conn_01x02, J501 54-00164, J502 5227699-1, J503 USB-B-S-X-X-VT, J504 Conn_01x06, J701 Conn_02x02_Odd_Even, J702 Conn_02x02_Odd_Even, J801 Conn_02x03_Odd_Even, SW701 PTS636SL43SMTRLFS, SW704 PTS636SL43SMTRLFS, U1001 NE555D, U1002 NE555D, U1003 TL082, U1004 TL082, U201 TL082, U202 TL082, U203 TL082, U204 TL082, U301 TL082, U302 TL082, U303 TL082, U304 TL082, U305 TL082, U401 LM311, U402 74LS08, U403 74AUC2G02, U404 74LS365, U501 REF102CU, U502 R-78E5.0-0.5, U503 TL082, U504 TL082, U505 TMH 0515D, U506 AMS1117-3.3, U701 74AUC2G02, U702 74LS32, U703 TL082, U704 TL082, U705 LM311

Commit message: updates board to REV 1 Ordered version
Parts:
- removed D506: 1N5819WS, Diode_SMD:D_SOD-323
- C203, C303: value 10uF 5% -> 10uF 10%
- C301, C302: value 27uF 5% -> 27nF 5%
- C501, C505, C508, C509, C510: value 10uF -> 10uF 10%
- C511: value 22uF -> 10uF 10%
- D501, D502, D704: value GREEN [XL-2012UGC] -> LTST-C170KGKT [GREEN]
- D503, D504, D505, D703: value RED [XL-2012SURC] -> LTST-C170KRKT [RED]
- R1004, R1005, R1009, R206, R207, R317, R502, R504, R702, R703, R704, R705, R706, R707, R708: value 10KΩ -> 10kΩ 1%
- R202, R210, R214, R215, R302, R308, R309, R310, R324, R325: value 10K -> 10kΩ 1%
- R209, R211, R213, R216, R217, R218, R219, R220, R307, R313, R316, R319, R322, R323, R326, R328, R329: value 10kΩ -> 10kΩ 1%
- SW701, SW704: value PTS636SL43SMTRLFS -> SW_PTS636S-J_CNK
- moved C405 384.6 mm to (443.0, 186.4)
- moved C701 360.4 mm to (444.8, 191.5), turned to 180 degrees
- moved U402 354.7 mm to (424.3, 186.7)
- moved U701 351.8 mm to (445.8, 189.0), turned to 180 degrees
- moved C712 350.4 mm to (442.3, 189.0), turned to -90 degrees
- moved C711 349.2 mm to (438.2, 195.6), turned to 90 degrees
- moved J701 341.3 mm to (431.3, 187.2)
- moved J702 341.3 mm to (431.3, 194.3)
- moved TP705 339.0 mm to (451.4, 200.7)
- moved R712 338.2 mm to (449.4, 189.3), turned to -90 degrees
- moved TP706 335.6 mm to (451.4, 194.3)
- moved C710 333.7 mm to (421.9, 193.0)
- moved C406 333.4 mm to (393.7, 171.4), turned to -90 degrees
- moved C407 333.4 mm to (393.4, 176.0), turned to -90 degrees
- moved C706 332.7 mm to (425.7, 170.3), turned to 180 degrees
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Connections:
- C510 pad 1: +5V -> +9V
- J503 pad 01: Net-(D506-K) -> +5V
- J801 pad 1: /Inner Current Regulator/D_Cmd -> /Int_Cmd
- J801 pad 3: /Int_Cmd -> /Ext_Cmd
- J801 pad 5: /Ext_Cmd -> /Inner Current Regulator/D_Cmd
- R314 pad 2: Net-(R314-Pad2) -> Net-(C301-Pad1)
- R318 pad 2: Net-(R314-Pad2) -> Net-(C301-Pad1)
- TP301 pad 1: Net-(R314-Pad2) -> Net-(C301-Pad1)
- U1004 pad 1: (no net) -> Net-(U1004A--)
- U1004 pad 2: (no net) -> Net-(U1004A--)
- U1004 pad 3: (no net) -> GND
- U304 pad 1: Net-(R314-Pad2) -> Net-(C301-Pad1)
- U403 pad 3: (no net) -> unconnected-(U403-Pad3)
- U403 pad 5: (no net) -> GND
- U403 pad 6: (no net) -> GND
- U504 pad 1: (no net) -> Net-(U504A--)
- U504 pad 2: (no net) -> Net-(U504A--)
- U504 pad 3: (no net) -> GND
- U506 pad 3: +5V -> +9V
- U702 pad 10: (no net) -> +5V
- U702 pad 11: (no net) -> unconnected-(U702-Pad11)
- U702 pad 12: (no net) -> +5V
- U702 pad 13: (no net) -> +5V
- U702 pad 4: (no net) -> +5V
- U702 pad 5: (no net) -> +5V
- U702 pad 6: (no net) -> unconnected-(U702-Pad6)
- U702 pad 8: (no net) -> unconnected-(U702-Pad8)
- U702 pad 9: (no net) -> +5V
- U704 pad 5: (no net) -> GND
- U704 pad 6: (no net) -> Net-(U704B--)
- U704 pad 7: (no net) -> Net-(U704B--)
Routing:
- net +15V: track 0.00 -> 804.5 mm, vias 0 -> 29
- net -15V: track 0.00 -> 712.8 mm, vias 0 -> 19
- net +5V: track 0.00 -> 611.0 mm, vias 0 -> 19
- net /+10V_Ref: track 0.00 -> 324.2 mm, vias 0 -> 7
- net /-10V_Ref: track 0.00 -> 263.5 mm, vias 0 -> 4
- net /I_Fdbk_Raw: track 0.00 -> 204.2 mm, vias 0 -> 3
- net /Modulator and Protection/Carrier Wave/Carrier: track 0.00 -> 182.8 mm
- net /Ext_Cmd: track 0.00 -> 179.3 mm, vias 0 -> 2
- net /V_Fdbk_Raw: track 0.00 -> 159.8 mm, vias 0 -> 2
- net /Int_Cmd: track 0.00 -> 135.9 mm, vias 0 -> 5
- net /Inner Current Regulator/I_Fdbk: track 0.00 -> 120.6 mm, vias 0 -> 4
- net /Inner Current Regulator/+I_Err: track 0.00 -> 106.2 mm, vias 0 -> 2
- net GND: track 0.00 -> 104.3 mm, vias 0 -> 112
- net +9V: track 0.00 -> 85.1 mm, vias 0 -> 3
- net /Modulator and Protection/Protection/Overcurrent: track 0.00 -> 82.5 mm, vias 0 -> 2
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- added copper zone on B.Cu, net GND
- added copper zone on F.Cu, net GND
Other:
- board size 228.6 x 81 mm -> 253.2 x 81 mm
- board text added: "! NON-STANDARD USB WIRING ! DO NOT CONNECT THIS PORT TO STANDARD USB HOSTS OR DEVICES The USB-B shell is wired with a non-standard pinout. Plugging in USB devices may cause permanent hardware damage"
- board text added: "+15V"
- board text added: "+5V"
- board text added: "+9V"
- board text added: "-15V"
- board text added: "-I"
- board text added: "-I_FDBK"
- board text added: "-P"
- board text added: "-R"
- board text added: "-V_FDBK"
- board text added: "3.3V"
- board text added: "D_CMD"
- board text added: "ERR"
- board text added: "EXT_CMD"
- board text added: "GND"
- board text added: "HB DRIVE V1"
- board text added: "IN: 9VDC >200mA"
- board text added: "INNER CURRENT REGULATOR"
- board text added: "INT_CMD"
- board text added: "I_CMD"
- board text added: "I_FDBK_RAW"
- board text added: "LATCH DIS"
- board text added: "LATCH EN"
- board text added: "MODULATION"
- board text added: "OK"
- board text added: "OUTER VOLTAGE REGULATOR"
- board text added: "OUTPUT AND SAFETY"
- board text added: "POWER AND INPUTS"
- board text added: "PROF. FLANNERY | MAX S | HUNTER K"
- board text added: "USR DIS"
- board text added: "USR RST"
- board text added: "V_FDBK_RAW"
- board text added: "WAVE 1"
- board text added: "WAVE 2"

Commit message: Annotates Schematic! Fixes REV1 wiring swaps and replaces buffer
Other:
- board text added: "OUTPUT AND PROTECTION"
- board text removed: "OUTPUT AND SAFETY"

Commit message: annotates PCB! wiring is still broken here
Parts:
- removed C1010, C1012: 10nF, Capacitor_SMD:C_0603_1608Metric_Pad1.08x0.95mm_HandSolder
- removed D1001, D1002: 1N4148W, Diode_SMD:D_SOD-123
- removed J1001: Conn_02x02_Odd_Even, Connector_PinHeader_2.54mm:PinHeader_2x02_P2.54mm_Vertical
- removed J402: Conn_01x02, Jumper:SolderJumper-2_P1.3mm_Open_TrianglePad1.0x1.5mm
- removed J504: Conn_01x06, Connector_PinHeader_2.54mm:PinHeader_1x06_P2.54mm_Vertical
- removed R1011: 680Ω, Resistor_SMD:R_0603_1608Metric_Pad0.98x0.95mm_HandSolder
- removed R1012: PV36W103C01B00, PV36W104C01B00:POT_PV36W_BRN
- removed R1013: 1KΩ, Resistor_SMD:R_0603_1608Metric_Pad0.98x0.95mm_HandSolder
- removed U1002: NE555D, Package_SO:SOIC-8_3.9x4.9mm_P1.27mm
- removed U701: 74AUC2G02, Package_SO:VSSOP-8_2.3x2mm_P0.5mm
- added C210: 100nF 100V, Capacitor_SMD:C_0603_1608Metric, F.Cu at (299.5, 182.9)
- added C211: 100nF 100V, Capacitor_SMD:C_0603_1608Metric, F.Cu at (302.6, 185.7)
- added C409: 100nF 100V, Capacitor_SMD:C_0603_1608Metric, F.Cu at (369.5, 203.7)
- added C410: 100nF 100V, Capacitor_SMD:C_0603_1608Metric, F.Cu at (363.6, 203.7)
- added J1002: Conn_02x04_Odd_Even, Connector_PinHeader_2.54mm:PinHeader_2x04_P2.54mm_Vertical, F.Cu at (363.4, 214.6)
- added J505: Conn_01x03, Connector_PinHeader_2.54mm:PinHeader_1x03_P2.54mm_Vertical, F.Cu at (212.9, 198.4)
- added J506: 3M_30306-6002HB, 30306_6002:30306-6002HB, F.Cu at (209.2, 185.7)
- added R221: 10kΩ 1%, Resistor_SMD:R_0603_1608Metric_Pad0.98x0.95mm_HandSolder, F.Cu at (293.2, 190.3)
- added R222: 10kΩ 1%, Resistor_SMD:R_0603_1608Metric_Pad0.98x0.95mm_HandSolder, F.Cu at (292.9, 185.4)
- added TP206: TestPoint, TestPoint:TestPoint_Loop_D2.60mm_Drill1.6mm_Beaded, F.Cu at (296.4, 176.7)
- added TP207: TestPoint, TestPoint:TestPoint_Loop_D2.60mm_Drill1.6mm_Beaded, F.Cu at (259.6, 187.5)
- added TP308: TestPoint, TestPoint:TestPoint_Loop_D2.60mm_Drill1.6mm_Beaded, F.Cu at (313.9, 185.9)
- added TP402: TestPoint, TestPoint:TestPoint_Loop_D2.60mm_Drill1.6mm_Beaded, F.Cu at (390.9, 193.5)
- added TP403: TestPoint, TestPoint:TestPoint_Loop_D2.60mm_Drill1.6mm_Beaded, F.Cu at (396.0, 193.8)
- added TP404: TestPoint, TestPoint:TestPoint_Loop_D2.60mm_Drill1.6mm_Beaded, F.Cu at (391.0, 198.7)
- added TP405: TestPoint, TestPoint:TestPoint_Loop_D2.60mm_Drill1.6mm_Beaded, F.Cu at (395.9, 198.6)
- added TP513: TestPoint, TestPoint:TestPoint_Loop_D2.60mm_Drill1.6mm_Beaded, F.Cu at (404.2, 161.7)
- added TP514: TestPoint, TestPoint:TestPoint_Loop_D2.60mm_Drill1.6mm_Beaded, F.Cu at (253.6, 171.9)
- added TP515: TestPoint, TestPoint:TestPoint_Loop_D2.60mm_Drill1.6mm_Beaded, F.Cu at (247.3, 164.1)
- added TP516: TestPoint, TestPoint:TestPoint_Loop_D2.60mm_Drill1.6mm_Beaded, F.Cu at (432.2, 208.1)
- added TP517: TestPoint, TestPoint:TestPoint_Loop_D2.60mm_Drill1.6mm_Beaded, F.Cu at (307.0, 184.6)
- added TP518: TestPoint, TestPoint:TestPoint_Loop_D2.60mm_Drill1.6mm_Beaded, F.Cu at (350.0, 166.3)
- added TP519: TestPoint, TestPoint:TestPoint_Loop_D2.60mm_Drill1.6mm_Beaded, F.Cu at (359.3, 175.4)
- added TP520: TestPoint, TestPoint:TestPoint_Loop_D2.60mm_Drill1.6mm_Beaded, F.Cu at (349.6, 224.1)
- added TP521: TestPoint, TestPoint:TestPoint_Loop_D2.60mm_Drill1.6mm_Beaded, F.Cu at (299.6, 213.6)
- added U205: TL082, Package_SO:SOIC-8_3.9x4.9mm_P1.27mm, F.Cu at (297.8, 186.5)
- added U405: 74AHC1GU04, Package_TO_SOT_SMD:SOT-23-5, F.Cu at (369.6, 207.1)
- added U406: 74AHC1G125, Package_TO_SOT_SMD:SOT-23-5, F.Cu at (365.1, 193.4)
- added U706: 74LS02, Package_SO:SOIC-14_3.9x8.7mm_P1.27mm, F.Cu at (444.7, 187.7)
- J203: value Conn_01x02 -> Conn_01x03; footprint Connector_PinHeader_1.27mm:PinHeader_1x02_P1.27mm_Vertical -> Connector_PinHeader_2.54mm:PinHeader_1x03_P2.54mm_Vertical
- J303: footprint Connector_PinHeader_1.27mm:PinHeader_1x02_P1.27mm_Vertical -> Connector_PinHeader_2.54mm:PinHeader_1x02_P2.54mm_Vertical
- J401: value Conn_01x02 -> Conn_01x03; footprint Jumper:SolderJumper-2_P1.3mm_Open_TrianglePad1.0x1.5mm -> Connector_PinHeader_2.54mm:PinHeader_1x03_P2.54mm_Vertical
- R1003, R1008, R201, R203, R204, R212, R301, R303, R306, R320, R327, R506, R701: value PV36W104C01B00 -> 100 kΩ
- R1007, R208, R321: value PV36W204C01B00 -> 200 kΩ
- R209, R323, R324, R325: value 10kΩ 1% -> 100kΩ 1%
- R316, R317: value 10kΩ 1% -> 5kΩ 1%
- R404, R405: value PV36W502C01B00 -> 5 kΩ
- U403: value 74AUC2G02 -> 74AHC1G125; footprint Package_SO:VSSOP-8_2.3x2mm_P0.5mm -> Package_TO_SOT_SMD:SOT-23-5
- U404: value 74LS365 -> 74AHC1GU04; footprint Package_SO:SOIC-16_3.9x9.9mm_P1.27mm -> Package_TO_SOT_SMD:SOT-23-5
- moved C702 70.5 mm to (449.4, 186.1), turned to 90 degrees
- moved U702 39.7 mm to (413.7, 198.0), turned to 0 degrees
- moved U403 39.4 mm to (363.7, 207.0)
- moved C701 36.9 mm to (408.1, 195.0), turned to -90 degrees
- moved J401 23.3 mm to (366.7, 198.8), turned to 90 degrees
- moved C404 20.8 mm to (364.5, 189.2), turned to 180 degrees
- moved TP708 18.6 mm to (404.7, 200.3)
- moved C1003 15.4 mm to (358.4, 213.5), turned to 180 degrees
- moved C1004 13.6 mm to (358.5, 222.5), turned to 180 degrees
- moved J203 13.3 mm to (301.0, 195.9), turned to 0 degrees
- moved TP704 13.0 mm to (404.3, 195.9)
- moved C408 13.0 mm to (364.5, 182.8), turned to 180 degrees
- moved C1002 11.1 mm to (358.4, 216.5), turned to 180 degrees
- moved R326 9.85 mm to (344.0, 188.2)
- moved C1006 8.06 mm to (386.9, 216.9)
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Connections:
- net /Modulator and Protection/Protection/Safety_Latch renamed /Modulator and Protection/Protection/Protection_Latch
- C1001 pad 1: Net-(U1001-THRES) -> Net-(J1002-Pin_5)
- C1002 pad 1: Net-(U1001-THRES) -> Net-(J1002-Pin_3)
- C1003 pad 1: Net-(U1001-THRES) -> Net-(J1002-Pin_1)
- C1004 pad 1: Net-(U1001-THRES) -> Net-(J1002-Pin_7)
- C1006 pad 2: Net-(J1001-Pin_2) -> Net-(U1001-OUT)
- C404 pad 1: GND -> +5V
- C404 pad 2: +5V -> GND
- C406 pad 1: /Modulator and Protection/Modulator and Dead Time Injector/HS_Buf_In -> Net-(C406-Pad1)
- C407 pad 1: /Modulator and Protection/Modulator and Dead Time Injector/LS_Buf_In -> Net-(C407-Pad1)
- C408 pad 1: GND -> +5V
- C408 pad 2: +5V -> GND
- J203 pad 1: Net-(J203-Pin_1) -> /Outer Voltage Regulator/+I_Cmd
- J401 pad 1: /Modulator and Protection/Modulator and Dead Time Injector/HS_Buf_Out -> Net-(J401-Pin_1)
- J401 pad 2: /Modulator and Protection/Modulator and Dead Time Injector/HS_Buf_In -> /Modulator and Protection/Modulator and Dead Time Injector/H_Cmd
- R1002 pad 2: Net-(U1001-THRES) -> /Modulator and Protection/Carrier Wave/Capacitor_Select
- R212 pad 2: Net-(J203-Pin_1) -> /Outer Voltage Regulator/-I_Cmd
- R212 pad 3: Net-(J203-Pin_1) -> /Outer Voltage Regulator/-I_Cmd
- R321 pad 2: /Inner Current Regulator/I_Fdbk -> /Inner Current Regulator/-I_Fdbk
- R321 pad 3: /Inner Current Regulator/I_Fdbk -> /Inner Current Regulator/-I_Fdbk
- R324 pad 1: Net-(J301-Pin_4) -> Net-(U305B--)
- R324 pad 2: Net-(U305B--) -> Net-(J301-Pin_4)
- R325 pad 1: Net-(J301-Pin_6) -> Net-(U305B--)
- R325 pad 2: Net-(U305B--) -> Net-(J301-Pin_6)
- R328 pad 2: /Inner Current Regulator/I_Fdbk -> /Inner Current Regulator/-I_Fdbk
- R403 pad 1: /Modulator and Protection/Modulator and Dead Time Injector/H_Cmd -> /Modulator and Protection/Modulator and Dead Time Injector/H_Cmd_Raw
- R404 pad 1: /Modulator and Protection/Modulator and Dead Time Injector/H_Cmd -> Net-(R404-Pad1)
- R404 pad 2: /Modulator and Protection/Modulator and Dead Time Injector/H_Cmd -> Net-(R404-Pad1)
- R406 pad 2: /Modulator and Protection/Modulator and Dead Time Injector/HS_Buf_In -> Net-(C406-Pad1)
- R407 pad 2: /Modulator and Protection/Modulator and Dead Time Injector/LS_Buf_In -> Net-(C407-Pad1)
- R408 pad 1: /Modulator and Protection/Modulator and Dead Time Injector/HS_Buf_In -> Net-(C406-Pad1)
- R409 pad 1: /Modulator and Protection/Modulator and Dead Time Injector/LS_Buf_In -> Net-(C407-Pad1)
- R702 pad 1: /Inner Current Regulator/I_Fdbk -> /Inner Current Regulator/-I_Fdbk
- TP1001 pad 1: Net-(J1001-Pin_3) -> Net-(U1001-OUT)
- TP202 pad 1: Net-(J203-Pin_1) -> /Outer Voltage Regulator/-I_Cmd
- TP305 pad 1: /Inner Current Regulator/I_Fdbk -> /Inner Current Regulator/-I_Fdbk
- TP401 pad 1: /Modulator and Protection/Modulator and Dead Time Injector/H_Cmd -> /Modulator and Protection/Modulator and Dead Time Injector/H_Cmd_Raw
- U1001 pad 2: Net-(U1001-THRES) -> /Modulator and Protection/Carrier Wave/Capacitor_Select
- U1001 pad 3: Net-(J1001-Pin_3) -> Net-(U1001-OUT)
- U1001 pad 6: Net-(U1001-THRES) -> /Modulator and Protection/Carrier Wave/Capacitor_Select
- U204 pad 7: Net-(J203-Pin_1) -> /Outer Voltage Regulator/-I_Cmd
- U301 pad 7: /Inner Current Regulator/I_Fdbk -> /Inner Current Regulator/-I_Fdbk
- U401 pad 7: /Modulator and Protection/Modulator and Dead Time Injector/H_Cmd -> /Modulator and Protection/Modulator and Dead Time Injector/H_Cmd_Raw
- U402 pad 1: /Modulator and Protection/Modulator and Dead Time Injector/H_Cmd -> Net-(R404-Pad1)
- U402 pad 10: /Modulator and Protection/Modulator and Dead Time Injector/G_Lower_Cmd -> /Modulator and Protection/Modulator and Dead Time Injector/G_Upper_Cmd
- U402 pad 13: /Modulator and Protection/Modulator and Dead Time Injector/G_Upper_Cmd -> /Modulator and Protection/Modulator and Dead Time Injector/G_Lower_Cmd
- U402 pad 14: GND -> +5V
- U402 pad 2: /Modulator and Protection/Modulator and Dead Time Injector/HS_Buf_Out -> Net-(C406-Pad1)
- U402 pad 5: /Modulator and Protection/Modulator and Dead Time Injector/LS_Buf_Out -> Net-(C407-Pad1)
- U402 pad 7: +5V -> GND
- U403 pad 1: /Modulator and Protection/Modulator and Dead Time Injector/H_Cmd -> unconnected-(U403-Pad1)
- U403 pad 3: unconnected-(U403-Pad3) -> GND
- U403 pad 4: +5V -> Net-(R404-Pad1)
- U403 pad 5: GND -> +5V
- U404 pad 1: GND -> unconnected-(U404-NC-Pad1)
- U404 pad 2: /Modulator and Protection/Modulator and Dead Time Injector/HS_Buf_In -> /Modulator and Protection/Modulator and Dead Time Injector/H_Cmd_Raw
- U404 pad 3: /Modulator and Protection/Modulator and Dead Time Injector/HS_Buf_Out -> GND
- U404 pad 4: GND -> Net-(J401-Pin_3)
- U404 pad 5: unconnected-(U404-O2-Pad5) -> +5V
Routing:
- net /Inner Current Regulator/I_Fdbk: track 120.6 -> 0.00 mm, vias 4 -> 0
- net /Inner Current Regulator/-I_Fdbk: track 0.00 -> 120.6 mm, vias 0 -> 4
- net (no net): track 0.00 -> 114.3 mm
- net /Modulator and Protection/Modulator and Dead Time Injector/HS_Buf_Out: track 64.3 -> 0.00 mm
- net Net-(C407-Pad1): track 0.00 -> 61.2 mm
- net /Modulator and Protection/Modulator and Dead Time Injector/LS_Buf_Out: track 61.2 -> 0.00 mm
- net +5V: track 611.0 -> 658.9 mm, vias 19 -> 15
- net Net-(U1001-OUT): track 0.00 -> 35.7 mm, vias 0 -> 1
- net /Modulator and Protection/Modulator and Dead Time Injector/LS_Buf_In: track 34.2 -> 0.00 mm
- net Net-(J203-Pin_1): track 33.9 -> 0.00 mm
- net /Outer Voltage Regulator/-I_Cmd: track 0.00 -> 33.9 mm
- net Net-(R405-Pad1): track 60.1 -> 92.8 mm, vias 1 -> 0
- net /Modulator and Protection/Modulator and Dead Time Injector/HS_Buf_In: track 27.4 -> 0.00 mm
- net Net-(U1001-THRES): track 25.8 -> 0.00 mm
- net Net-(J1001-Pin_3): track 20.4 -> 0.00 mm, vias 1 -> 0
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Other:
- board size 253.2 x 81 mm -> 253.2 x 77 mm
- board text added: "+10V"
- board text added: "+I_Err"
- board text added: "+I_Fdbk"
- board text added: "+Res_Reg_Cmd"
- board text added: "+V_Err"
- board text added: "+V_Fdbk"
- board text added: "-10V"
- board text added: "-I_Err"
- board text added: "-I_Fdbk"
- board text added: "-Res_Reg_Cmd"
- board text added: "-V_Err"
- board text added: "-V_Fdbk"
- board text added: "Bipolar Triangle Wave"
- board text added: "Carrier"
- board text added: "DC Offset"
- board text added: "DIS"
- board text added: "D_Cmd"
- board text added: "Err"
- board text added: "Ext_Cmd"
- board text added: "G_Lower"
- board text added: "G_Upper"
- board text added: "Gain"
- board text added: "Gain In"
- board text added: "Gain Out"
- board text added: "H"
- board text added: "H+RC"
- board text added: "H_Cmd_Raw"
- board text added: "I_Abs"
- board text added: "I_Limit"
- board text added: "Int DC Ref"
- board text added: "Integral"
- board text added: "Integrator In"
- board text added: "Latch"
- board text added: "Lower RC"
- board text added: "Overcurrent"
- board text added: "Proportional"
- board text added: "Raw Square Wave"
- board text added: "Resonant"
- board text added: "Square Wave with DC Blocking"
- board text added: "Upper RC"
- board text removed: "I_FDBK_RAW"
- board text removed: "V_FDBK_RAW"
- board text removed: "WAVE 1"
- board text removed: "WAVE 2"

Commit message: Preliminary wiring of V2 completed, yet to pass DRC
Parts:
- moved C405 16.7 mm to (426.2, 181.2)
- moved C210 7.81 mm to (297.4, 190.4), turned to 0 degrees
- moved J505 5.13 mm to (207.7, 198.4), turned to 90 degrees
- moved TP514 4.72 mm to (252.2, 176.4)
- moved J303 1.31 mm to (348.6, 185.8)
- moved TP1001 0.74 mm to (370.8, 214.4)
- moved TP1004 0.64 mm to (398.4, 208.3)
- turned R324 to 180 degrees
- turned R325 to 180 degrees
Routing:
- net (no net): track 114.3 -> 0.04 mm
- net Net-(R404-Pad1): track 4.18 -> 116.0 mm, vias 0 -> 1
- net GND: track 100.3 -> 34.2 mm, vias 99 -> 479
- net +15V: track 804.5 -> 867.9 mm, vias 26 -> 35
- net /Modulator and Protection/Modulator and Dead Time Injector/H_Cmd_Raw: track 0.00 -> 56.1 mm, vias 0 -> 1
- net /Modulator and Protection/Modulator and Dead Time Injector/H_Cmd: track 72.2 -> 16.7 mm
- net Net-(C406-Pad1): track 0.00 -> 55.0 mm, vias 0 -> 1
- net /Modulator and Protection/Carrier Wave/Capacitor_Select: track 0.00 -> 35.9 mm
- net /Modulator and Protection/Protection/Overcurrent: track 79.8 -> 48.2 mm
- net Net-(R711-Pad1): track 61.0 -> 30.9 mm
- net Net-(R710-Pad2): track 55.8 -> 27.2 mm, vias 2 -> 4
- net /Outer Voltage Regulator/+I_Cmd: track 0.00 -> 25.0 mm
- net /Inner Current Regulator/-I_Fdbk: track 120.6 -> 144.5 mm
- net +5V: track 658.9 -> 638.1 mm, vias 15 -> 24
- net /V_Fdbk_Raw: track 159.8 -> 140.1 mm
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