File: HB_Drive_V1/HB_Drive_V1.kicad_pcb (KiCad board)
At the start: 2 copper layers, 253.2 x 77 mm, 277 parts, among them J1002 Conn_02x04_Odd_Even, J201 Conn_02x02_Odd_Even, J202 Conn_02x03_Odd_Even, J203 Conn_01x03, J301 Conn_02x03_Odd_Even, J304 Conn_02x04_Odd_Even, J401 Conn_01x03, J501 54-00164, J502 5227699-1, J503 USB-B-S-X-X-VT, J505 Conn_01x03, J506 30306-6002HB, J701 Conn_02x02_Odd_Even, J702 Conn_02x02_Odd_Even, J801 Conn_02x03_Odd_Even, Q701 BSS138, Q702 BSS138, SW701 PTS636SL43SMTRLFS, SW704 PTS636SL43SMTRLFS, U1001 NE555D, U1003 TL082, U1004 TL082, U201 TL082, U202 TL082, U203 TL082, U204 TL082, U205 TL082, U301 TL082, U302 TL082, U303 TL082, U304 TL082, U305 TL082, U401 LM311, U402 74LS08, U403 74AHC1G125, U404 74AHC1GU04, U405 74AHC1GU04, U406 74AHC1G125, U501 REF102AU, U502 R-78E5.0-0.5, U503 TL082, U504 TL082, U505 TMH 0515D, U506 AMS1117-3.3, U702 74LS32, U703 TL082, U704 TL082, U705 LM311, U706 74LS02

Commit message: Brings everything up to latest copy on my computer
Parts:
- added C314: 200pF 50V, Capacitor_SMD:C_0603_1608Metric, F.Cu at (331.5, 178.2)
- added TP208: TestPoint, TestPoint:TestPoint_Loop_D2.60mm_Drill1.6mm_Beaded, F.Cu at (301.1, 212.9)
- added TP209: TestPoint, TestPoint:TestPoint_Loop_D2.60mm_Drill1.6mm_Beaded, F.Cu at (301.1, 218.3)
- added TP309: TestPoint, TestPoint:TestPoint_Loop_D2.60mm_Drill1.6mm_Beaded, F.Cu at (350.5, 217.8)
- added TP310: TestPoint, TestPoint:TestPoint_Loop_D2.60mm_Drill1.6mm_Beaded, F.Cu at (350.5, 213.5)
- R321: value 200 kΩ -> 500 kΩ
- moved TP520 39.9 mm to (309.7, 223.3)
- moved TP521 30.1 mm to (269.5, 214.8)
- moved TP303 10.1 mm to (350.5, 222.1)
- moved TP512 9.72 mm to (226.0, 176.0)
- moved C705 6.40 mm to (404.4, 183.2), turned to 0 degrees
- moved C312 6.37 mm to (332.2, 185.6)
- moved C206 5.98 mm to (266.4, 186.0), turned to 180 degrees
- moved R206 5.43 mm to (261.5, 191.2)
- moved R405 5.42 mm to (381.8, 185.3)
- moved C1011 4.77 mm to (419.0, 216.9)
- moved TP1003 4.46 mm to (426.8, 213.5)
- moved TP516 2.66 mm to (432.0, 209.2)
- moved R404 2.61 mm to (381.6, 176.5)
- moved TP1002 2.54 mm to (392.9, 214.2)
- moved TP701 1.79 mm to (404.1, 177.8)
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Routing:
- net /Outer Voltage Regulator/-Int_Reg_Cmd: track 14.0 -> 43.4 mm
- net /Outer Voltage Regulator/-Prop_Reg_Cmd: track 30.3 -> 59.2 mm
- net /Inner Current Regulator/-Prop_Reg_Cmd: track 27.1 -> 54.0 mm, vias 0 -> 1
- net /Inner Current Regulator/-Int_Reg_Cmd: track 15.9 -> 42.6 mm
- net /Inner Current Regulator/-Res_Reg_Cmd: track 51.5 -> 66.7 mm
- net -15V: track 722.9 -> 736.1 mm
- net /V_Fdbk_Raw: track 313.2 -> 302.1 mm
- net Net-(U301B--): track 24.5 -> 31.4 mm
- net +15V: track 868.0 -> 861.6 mm
- net /Modulator and Protection/Carrier Wave/Carrier: track 167.7 -> 172.0 mm
- net Net-(R404-Pad1): track 116.0 -> 119.4 mm
- net Net-(U201B--): track 24.5 -> 27.9 mm
- net +5V: track 638.8 -> 641.7 mm
- net Net-(C1006-Pad1): track 17.3 -> 20.0 mm
- net Net-(R405-Pad3): track 6.75 -> 8.89 mm
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Other:
- outline, holes or cut-outs redrawn
- board text added: "-Int_Reg_Cmd"
- board text added: "-Prop_Reg_Cmd"
- board text added: "Gate Control"
- board text added: "NON-STANDARD USB WIRING DO NOT CONNECT THIS PORT TO STANDARD USB HOSTS OR DEVICES The USB-B shell is wired with a non-standard pinout. Plugging in USB devices may cause permanent hardware damage"
- board text added: "V/I Sense"
- board text removed: "! NON-STANDARD USB WIRING ! DO NOT CONNECT THIS PORT TO STANDARD USB HOSTS OR DEVICES The USB-B shell is wired with a non-standard pinout. Plugging in USB devices may cause permanent hardware damage"
- board text removed: "Int DC Ref"
