File: HB_Drive_V1/Modulator.kicad_sch (KiCad schematic)
At the start: 1 part, among them J801 Conn_02x03_Odd_Even

Commit message: restores v2 to condtion as ordered!
Connections:
- net Modulator and Dead Time Injector/D_Cmd renamed Modulator and Dead Time Injector/Duty
Other:
- sheet Modulator and Dead Time Injector ports: added Duty; removed D_Cmd
Changed lines of the file:
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@@
 			)
 		)
-		(pin "D_Cmd" input
+		(pin "Duty" input
 			(at 101.6 76.2 180)
 			(effects

Commit message: Brings everything up to latest copy on my computer
Other:
- company: (none) -> UW Madison, WEMPEC
- title: (none) -> HB Drive V3
Changed lines of the file:
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@@
 	(generator_version "10.0")
 	(paper "A4")
+	(title_block
+		(title "HB Drive V3")
+		(date "2026-09-08")
+		(company "UW Madison, WEMPEC")
+	)
 	(junction
 		(at 95.25 76.2)
